Commit message: Intecremental updates
Signed-off-by: SteveMacenski <stevenmacenski@gmail.com>

File: opennav_benchmark_sim/worlds/benchmark_warehouse.sdf.xacro (robot description, xacro)
@@ -4,7 +4,7 @@
   <world name="benchmark_warehouse">
     <!-- Physics -->
-    <physics name="3ms" type="ode">
-      <max_step_size>0.003</max_step_size>
-      <real_time_update_rate>1000.0</real_time_update_rate>
+    <physics name="5ms" type="bullet">
+      <max_step_size>0.005</max_step_size>
+      <real_time_update_rate>500.0</real_time_update_rate>
       <real_time_factor>1.0</real_time_factor>
     </physics>
@@ -40,23 +40,13 @@
       <direction>-0.3 0.2 -1.0</direction>
     </light>
-    <!-- Ground plane (matches wall dimensions: 120m x 155m) -->
+    <!-- Ground plane (120m x 140m) -->
     <model name="ground_plane">
       <static>true</static>
       <link name="link">
         <collision name="collision">
-          <geometry>
-            <plane>
-              <normal>0 0 1</normal>
-              <size>120 155</size>
-            </plane>
-          </geometry>
+          <geometry><plane><normal>0 0 1</normal><size>120 140</size></plane></geometry>
         </collision>
         <visual name="visual">
-          <geometry>
-            <plane>
-              <normal>0 0 1</normal>
-              <size>120 155</size>
-            </plane>
-          </geometry>
+          <geometry><plane><normal>0 0 1</normal><size>120 140</size></plane></geometry>
           <material>
             <ambient>0.55 0.55 0.53 1</ambient>
@@ -69,7 +59,7 @@
     </model>
     <!-- ============================================================ -->
-    <!-- PERIMETER WALLS (120m x 155m, 5m tall)                       -->
-    <!-- Two-tone: dark concrete base (1.5m) + metal upper (3.5m)     -->
-    <!-- ============================================================ -->
+    <!-- MACROS                                                        -->
+    <!-- ============================================================ -->
+    <!-- Brick perimeter wall (10.0m tall, two-tone red brick) -->
     <xacro:macro name="wall_segment" params="name x y yaw length">
       <model name="wall_${name}">
@@ -78,97 +68,102 @@
         <link name="link">
           <visual name="lower">
-            <pose>0 0 0.75 0 0 0</pose>
-            <geometry>
-              <box><size>${length} 0.3 1.5</size></box>
-            </geometry>
+            <pose>0 0 1.25 0 0 0</pose>
+            <geometry><box><size>${length} 0.3 2.5</size></box></geometry>
             <material>
-              <ambient>0.4 0.4 0.42 1</ambient>
-              <diffuse>0.4 0.4 0.42 1</diffuse>
-              <specular>0.1 0.1 0.1 1</specular>
+              <ambient>0.50 0.18 0.08 1</ambient>
+              <diffuse>0.50 0.18 0.08 1</diffuse>
+              <specular>0.05 0.05 0.05 1</specular>
             </material>
           </visual>
           <visual name="upper">
-            <pose>0 0 3.25 0 0 0</pose>
-            <geometry>
-              <box><size>${length} 0.3 3.5</size></box>
-            </geometry>
+            <pose>0 0 6.25 0 0 0</pose>
+            <geometry><box><size>${length} 0.3 7.5</size></box></geometry>
             <material>
-              <ambient>0.678 0.678 0.678 1</ambient>
-              <diffuse>0.678 0.678 0.678 1</diffuse>
-              <specular>0.3 0.3 0.3 1</specular>
+              <ambient>0.65 0.28 0.12 1</ambient>
+              <diffuse>0.65 0.28 0.12 1</diffuse>
+              <specular>0.05 0.05 0.05 1</specular>
+            </material>
+          </visual>
+          <collision name="collision">
+            <pose>0 0 5.0 0 0 0</pose>
+            <geometry><box><size>${length} 0.3 10.0</size></box></geometry>
+          </collision>
+        </link>
+      </model>
+    </xacro:macro>
+    <!-- Roll-up dock door (4m wide x 5m tall, brick above) -->
+    <xacro:macro name="dock_door" params="name x y yaw">
+      <model name="door_${name}">
+        <static>true</static>
+        <pose>${x} ${y} 0 0 0 ${yaw}</pose>
+        <link name="link">
+          <visual name="door_panel">
+            <pose>0 0 2.5 0 0 0</pose>
+            <geometry><box><size>4.0 0.15 5.0</size></box></geometry>
+            <material>
+              <ambient>0.55 0.56 0.58 1</ambient>
+              <diffuse>0.55 0.56 0.58 1</diffuse>
+              <specular>0.4 0.4 0.4 1</specular>
+            </material>
+          </visual>
+          <visual name="above_door">
+            <pose>0 0 7.5 0 0 0</pose>
+            <geometry><box><size>4.0 0.3 5.0</size></box></geometry>
+            <material>
+              <ambient>0.65 0.28 0.12 1</ambient>
+              <diffuse>0.65 0.28 0.12 1</diffuse>
+              <specular>0.05 0.05 0.05 1</specular>
             </material>
           </visual>
           <collision name="collision">
             <pose>0 0 2.5 0 0 0</pose>
-            <geometry>
-              <box><size>${length} 0.3 5.0</size></box>
-            </geometry>
+            <geometry><box><size>4.0 0.15 5.0</size></box></geometry>
           </collision>
         </link>
       </model>
     </xacro:macro>
-    <xacro:wall_segment name="north" x="0" y="77.5" yaw="0" length="120"/>
-    <xacro:wall_segment name="south" x="0" y="-77.5" yaw="0" length="120"/>
-    <xacro:wall_segment name="east" x="60" y="0" yaw="1.5708" length="155"/>
-    <xacro:wall_segment name="west" x="-60" y="0" yaw="1.5708" length="155"/>
-    <!-- Support columns every 15m along walls -->
+    <!-- Support column (10.0m tall) -->
     <xacro:macro name="support_column" params="name x y">
-      <model name="column_${name}">
+      <model name="col_${name}">
         <static>true</static>
-        <pose>${x} ${y} 2.5 0 0 0</pose>
+        <pose>${x} ${y} 5.0 0 0 0</pose>
         <link name="link">
           <visual name="visual">
-            <geometry>
-              <box><size>0.4 0.4 5.0</size></box>
-            </geometry>
+            <geometry><box><size>0.4 0.4 10.0</size></box></geometry>
             <material>
-              <ambient>0.5 0.5 0.55 1</ambient>
-              <diffuse>0.5 0.5 0.55 1</diffuse>
+              <ambient>0.55 0.52 0.50 1</ambient>
+              <diffuse>0.55 0.52 0.50 1</diffuse>
               <specular>0.2 0.2 0.2 1</specular>
             </material>
           </visual>
           <collision name="collision">
-            <geometry>
-              <box><size>0.4 0.4 5.0</size></box>
-            </geometry>
+            <geometry><box><size>0.4 0.4 10.0</size></box></geometry>
           </collision>
         </link>
       </model>
     </xacro:macro>
-    <!-- North/South wall columns -->
-    <xacro:support_column name="n1" x="-45" y="77.5"/>
-    <xacro:support_column name="n2" x="-30" y="77.5"/>
-    <xacro:support_column name="n3" x="-15" y="77.5"/>
-    <xacro:support_column name="n4" x="0" y="77.5"/>
-    <xacro:support_column name="n5" x="15" y="77.5"/>
-    <xacro:support_column name="n6" x="30" y="77.5"/>
-    <xacro:support_column name="n7" x="45" y="77.5"/>
-    <xacro:support_column name="s1" x="-45" y="-77.5"/>
-    <xacro:support_column name="s2" x="-30" y="-77.5"/>
-    <xacro:support_column name="s3" x="-15" y="-77.5"/>
-    <xacro:support_column name="s4" x="0" y="-77.5"/>
-    <xacro:support_column name="s5" x="15" y="-77.5"/>
-    <xacro:support_column name="s6" x="30" y="-77.5"/>
-    <xacro:support_column name="s7" x="45" y="-77.5"/>
-    <!-- East/West wall columns -->
-    <xacro:support_column name="e1" x="60" y="-60"/>
-    <xacro:support_column name="e2" x="60" y="-30"/>
-    <xacro:support_column name="e3" x="60" y="0"/>
-    <xacro:support_column name="e4" x="60" y="30"/>
-    <xacro:support_column name="e5" x="60" y="60"/>
-    <xacro:support_column name="w1" x="-60" y="-60"/>
-    <xacro:support_column name="w2" x="-60" y="-30"/>
-    <xacro:support_column name="w3" x="-60" y="0"/>
-    <xacro:support_column name="w4" x="-60" y="30"/>
-    <xacro:support_column name="w5" x="-60" y="60"/>
-    <!-- ============================================================ -->
-    <!-- SHELF MACROS                                                  -->
-    <!-- All shelves rotated 90deg (yaw=1.5708) so long axis is N-S   -->
-    <!-- shelf: ~3.5m long x ~1m deep -> rotated: ~1m in X, ~3.5m in Y-->
-    <!-- shelf_big: ~7.5m long x ~1.2m deep -> rotated: ~1.2m X, ~7.5m Y -->
-    <!-- ============================================================ -->
+    <!-- Shelf macros: ALL running E-W (long axis in X), yaw=0 -->
+    <!-- shelf default: 3.5m X x 1m Y -->
     <xacro:macro name="small_shelf" params="name x y">
       <include>
-        <uri>https://fuel.gazebosim.org/1.0/MovAi/models/shelf</uri>
+        <uri>shelf</uri>
+        <name>${name}</name>
+        <pose>${x} ${y} 0 0 0 0</pose>
+        <static>true</static>
+      </include>
+    </xacro:macro>
+    <!-- shelf_big default: 7.5m X x 1.2m Y -->
+    <xacro:macro name="big_shelf" params="name x y">
+      <include>
+        <uri>shelf_big</uri>
+        <name>${name}</name>
+        <pose>${x} ${y} 0 0 0 0</pose>
+        <static>true</static>
+      </include>
+    </xacro:macro>
+    <!-- shelf_big rotated N-S: 1.2m X x 7.5m Y -->
+    <xacro:macro name="big_shelf_ns" params="name x y">
+      <include>
+        <uri>shelf_big</uri>
         <name>${name}</name>
         <pose>${x} ${y} 0 0 0 1.5708</pose>
@@ -176,451 +171,1016 @@
       </include>
     </xacro:macro>
-    <xacro:macro name="big_shelf" params="name x y">
+    <!-- Pallet macro -->
+    <xacro:macro name="pallet" params="name x y z yaw">
       <include>
-        <uri>https://fuel.gazebosim.org/1.0/MovAi/models/shelf_big</uri>
+        <uri>pallet_box_mobile</uri>
         <name>${name}</name>
-        <pose>${x} ${y} 0 0 0 1.5708</pose>
+        <pose>${x} ${y} ${z} 0 0 ${yaw}</pose>
         <static>true</static>
       </include>
     </xacro:macro>
     <!-- ============================================================ -->
-    <!-- ZONE A: HIGH-DENSITY (small shelves, 2.5m aisles)            -->
-    <!-- x=-55 to -17, 8 rows, center-to-center 5m in X              -->
-    <!-- Shelf ~1m wide rotated + 2.5m aisle -> NOT overlapping but   -->
-    <!-- the models may be wider; using 5m spacing to be safe         -->
-    <!-- Upper: y=+35 to +63, Lower: y=+8 to +28                     -->
-    <!-- Shelves placed ~4m apart in Y (each ~3.5m long rotated)      -->
-    <!-- ============================================================ -->
-    <!-- Zone A Upper (y=+35 to +63): 8 rows, 7 shelves per row in Y -->
-    <xacro:small_shelf name="za_r1_u1" x="-55" y="36"/>
-    <xacro:small_shelf name="za_r1_u2" x="-55" y="40"/>
-    <xacro:small_shelf name="za_r1_u3" x="-55" y="44"/>
-    <xacro:small_shelf name="za_r1_u4" x="-55" y="48"/>
-    <xacro:small_shelf name="za_r1_u5" x="-55" y="52"/>
-    <xacro:small_shelf name="za_r1_u6" x="-55" y="56"/>
-    <xacro:small_shelf name="za_r1_u7" x="-55" y="60"/>
-    <xacro:small_shelf name="za_r2_u1" x="-50" y="36"/>
-    <xacro:small_shelf name="za_r2_u2" x="-50" y="40"/>
-    <xacro:small_shelf name="za_r2_u3" x="-50" y="44"/>
-    <xacro:small_shelf name="za_r2_u4" x="-50" y="48"/>
-    <xacro:small_shelf name="za_r2_u5" x="-50" y="52"/>
-    <xacro:small_shelf name="za_r2_u6" x="-50" y="56"/>
-    <xacro:small_shelf name="za_r2_u7" x="-50" y="60"/>
-    <xacro:small_shelf name="za_r3_u1" x="-45" y="36"/>
-    <xacro:small_shelf name="za_r3_u2" x="-45" y="40"/>
-    <xacro:small_shelf name="za_r3_u3" x="-45" y="44"/>
-    <xacro:small_shelf name="za_r3_u4" x="-45" y="48"/>
-    <xacro:small_shelf name="za_r3_u5" x="-45" y="52"/>
-    <xacro:small_shelf name="za_r3_u6" x="-45" y="56"/>
-    <xacro:small_shelf name="za_r3_u7" x="-45" y="60"/>
-    <xacro:small_shelf name="za_r4_u1" x="-40" y="36"/>
-    <xacro:small_shelf name="za_r4_u2" x="-40" y="40"/>
-    <xacro:small_shelf name="za_r4_u3" x="-40" y="44"/>
-    <xacro:small_shelf name="za_r4_u4" x="-40" y="48"/>
-    <xacro:small_shelf name="za_r4_u5" x="-40" y="52"/>
-    <xacro:small_shelf name="za_r4_u6" x="-40" y="56"/>
-    <xacro:small_shelf name="za_r4_u7" x="-40" y="60"/>
-    <xacro:small_shelf name="za_r5_u1" x="-35" y="36"/>
-    <xacro:small_shelf name="za_r5_u2" x="-35" y="40"/>
-    <xacro:small_shelf name="za_r5_u3" x="-35" y="44"/>
-    <xacro:small_shelf name="za_r5_u4" x="-35" y="48"/>
-    <xacro:small_shelf name="za_r5_u5" x="-35" y="52"/>
-    <xacro:small_shelf name="za_r5_u6" x="-35" y="56"/>
-    <xacro:small_shelf name="za_r5_u7" x="-35" y="60"/>
-    <xacro:small_shelf name="za_r6_u1" x="-30" y="36"/>
-    <xacro:small_shelf name="za_r6_u2" x="-30" y="40"/>
-    <xacro:small_shelf name="za_r6_u3" x="-30" y="44"/>
-    <xacro:small_shelf name="za_r6_u4" x="-30" y="48"/>
-    <xacro:small_shelf name="za_r6_u5" x="-30" y="52"/>
-    <xacro:small_shelf name="za_r6_u6" x="-30" y="56"/>
-    <xacro:small_shelf name="za_r6_u7" x="-30" y="60"/>
-    <xacro:small_shelf name="za_r7_u1" x="-25" y="36"/>
-    <xacro:small_shelf name="za_r7_u2" x="-25" y="40"/>
-    <xacro:small_shelf name="za_r7_u3" x="-25" y="44"/>
-    <xacro:small_shelf name="za_r7_u4" x="-25" y="48"/>
-    <xacro:small_shelf name="za_r7_u5" x="-25" y="52"/>
-    <xacro:small_shelf name="za_r7_u6" x="-25" y="56"/>
-    <xacro:small_shelf name="za_r7_u7" x="-25" y="60"/>
-    <xacro:small_shelf name="za_r8_u1" x="-20" y="36"/>
-    <xacro:small_shelf name="za_r8_u2" x="-20" y="40"/>
-    <xacro:small_shelf name="za_r8_u3" x="-20" y="44"/>
-    <xacro:small_shelf name="za_r8_u4" x="-20" y="48"/>
-    <xacro:small_shelf name="za_r8_u5" x="-20" y="52"/>
-    <xacro:small_shelf name="za_r8_u6" x="-20" y="56"/>
-    <xacro:small_shelf name="za_r8_u7" x="-20" y="60"/>
-    <!-- Zone A Lower (y=+8 to +28): 8 rows, 5 shelves per row -->
-    <xacro:small_shelf name="za_r1_l1" x="-55" y="10"/>
-    <xacro:small_shelf name="za_r1_l2" x="-55" y="14"/>
-    <xacro:small_shelf name="za_r1_l3" x="-55" y="18"/>
-    <xacro:small_shelf name="za_r1_l4" x="-55" y="22"/>
-    <xacro:small_shelf name="za_r1_l5" x="-55" y="26"/>
-    <xacro:small_shelf name="za_r2_l1" x="-50" y="10"/>
-    <xacro:small_shelf name="za_r2_l2" x="-50" y="14"/>
-    <xacro:small_shelf name="za_r2_l3" x="-50" y="18"/>
-    <xacro:small_shelf name="za_r2_l4" x="-50" y="22"/>
-    <xacro:small_shelf name="za_r2_l5" x="-50" y="26"/>
-    <xacro:small_shelf name="za_r3_l1" x="-45" y="10"/>
-    <xacro:small_shelf name="za_r3_l2" x="-45" y="14"/>
-    <xacro:small_shelf name="za_r3_l3" x="-45" y="18"/>
-    <xacro:small_shelf name="za_r3_l4" x="-45" y="22"/>
-    <xacro:small_shelf name="za_r3_l5" x="-45" y="26"/>
-    <xacro:small_shelf name="za_r4_l1" x="-40" y="10"/>
-    <xacro:small_shelf name="za_r4_l2" x="-40" y="14"/>
-    <xacro:small_shelf name="za_r4_l3" x="-40" y="18"/>
-    <xacro:small_shelf name="za_r4_l4" x="-40" y="22"/>
-    <xacro:small_shelf name="za_r4_l5" x="-40" y="26"/>
-    <xacro:small_shelf name="za_r5_l1" x="-35" y="10"/>
-    <xacro:small_shelf name="za_r5_l2" x="-35" y="14"/>
-    <xacro:small_shelf name="za_r5_l3" x="-35" y="18"/>
-    <xacro:small_shelf name="za_r5_l4" x="-35" y="22"/>
-    <xacro:small_shelf name="za_r5_l5" x="-35" y="26"/>
-    <xacro:small_shelf name="za_r6_l1" x="-30" y="10"/>
-    <xacro:small_shelf name="za_r6_l2" x="-30" y="14"/>
-    <xacro:small_shelf name="za_r6_l3" x="-30" y="18"/>
-    <xacro:small_shelf name="za_r6_l4" x="-30" y="22"/>
-    <xacro:small_shelf name="za_r6_l5" x="-30" y="26"/>
-    <xacro:small_shelf name="za_r7_l1" x="-25" y="10"/>
-    <xacro:small_shelf name="za_r7_l2" x="-25" y="14"/>
-    <xacro:small_shelf name="za_r7_l3" x="-25" y="18"/>
-    <xacro:small_shelf name="za_r7_l4" x="-25" y="22"/>
-    <xacro:small_shelf name="za_r7_l5" x="-25" y="26"/>
-    <xacro:small_shelf name="za_r8_l1" x="-20" y="10"/>
-    <xacro:small_shelf name="za_r8_l2" x="-20" y="14"/>
-    <xacro:small_shelf name="za_r8_l3" x="-20" y="18"/>
-    <xacro:small_shelf name="za_r8_l4" x="-20" y="22"/>
-    <xacro:small_shelf name="za_r8_l5" x="-20" y="26"/>
-    <!-- ============================================================ -->
-    <!-- ZONE B: STANDARD (big shelves, 3.5m aisles)                  -->
-    <!-- x=-10 to +55, 10 rows, center-to-center 7m in X             -->
-    <!-- shelf_big ~1.2m wide rotated + 3.5m aisle, 7m safe spacing  -->
-    <!-- Upper: y=+35 to +63, Lower: y=+8 to +28                     -->
-    <!-- Shelves ~8m apart in Y (each ~7.5m long rotated)             -->
-    <!-- ============================================================ -->
-    <!-- Zone B Upper (y=+35 to +63): 10 rows, 3 shelves per row -->
-    <xacro:big_shelf name="zb_r1_u1" x="-10" y="39"/>
-    <xacro:big_shelf name="zb_r1_u2" x="-10" y="47"/>
-    <xacro:big_shelf name="zb_r1_u3" x="-10" y="55"/>
-    <xacro:big_shelf name="zb_r2_u1" x="-3" y="39"/>
-    <xacro:big_shelf name="zb_r2_u2" x="-3" y="47"/>
-    <xacro:big_shelf name="zb_r2_u3" x="-3" y="55"/>
-    <xacro:big_shelf name="zb_r3_u1" x="4" y="39"/>
-    <xacro:big_shelf name="zb_r3_u2" x="4" y="47"/>
-    <xacro:big_shelf name="zb_r3_u3" x="4" y="55"/>
-    <xacro:big_shelf name="zb_r4_u1" x="11" y="39"/>
-    <xacro:big_shelf name="zb_r4_u2" x="11" y="47"/>
-    <xacro:big_shelf name="zb_r4_u3" x="11" y="55"/>
-    <xacro:big_shelf name="zb_r5_u1" x="18" y="39"/>
-    <xacro:big_shelf name="zb_r5_u2" x="18" y="47"/>
-    <xacro:big_shelf name="zb_r5_u3" x="18" y="55"/>
-    <xacro:big_shelf name="zb_r6_u1" x="25" y="39"/>
-    <xacro:big_shelf name="zb_r6_u2" x="25" y="47"/>
-    <xacro:big_shelf name="zb_r6_u3" x="25" y="55"/>
-    <xacro:big_shelf name="zb_r7_u1" x="32" y="39"/>
-    <xacro:big_shelf name="zb_r7_u2" x="32" y="47"/>
-    <xacro:big_shelf name="zb_r7_u3" x="32" y="55"/>
-    <xacro:big_shelf name="zb_r8_u1" x="39" y="39"/>
-    <xacro:big_shelf name="zb_r8_u2" x="39" y="47"/>
-    <xacro:big_shelf name="zb_r8_u3" x="39" y="55"/>
-    <xacro:big_shelf name="zb_r9_u1" x="46" y="39"/>
-    <xacro:big_shelf name="zb_r9_u2" x="46" y="47"/>
-    <xacro:big_shelf name="zb_r9_u3" x="46" y="55"/>
-    <xacro:big_shelf name="zb_r10_u1" x="53" y="39"/>
-    <xacro:big_shelf name="zb_r10_u2" x="53" y="47"/>
-    <xacro:big_shelf name="zb_r10_u3" x="53" y="55"/>
-    <!-- Zone B Lower (y=+8 to +28): 10 rows, 2 shelves per row -->
-    <xacro:big_shelf name="zb_r1_l1" x="-10" y="12"/>
-    <xacro:big_shelf name="zb_r1_l2" x="-10" y="20"/>
-    <xacro:big_shelf name="zb_r2_l1" x="-3" y="12"/>
-    <xacro:big_shelf name="zb_r2_l2" x="-3" y="20"/>
-    <xacro:big_shelf name="zb_r3_l1" x="4" y="12"/>
-    <xacro:big_shelf name="zb_r3_l2" x="4" y="20"/>
-    <xacro:big_shelf name="zb_r4_l1" x="11" y="12"/>
-    <xacro:big_shelf name="zb_r4_l2" x="11" y="20"/>
-    <xacro:big_shelf name="zb_r5_l1" x="18" y="12"/>
-    <xacro:big_shelf name="zb_r5_l2" x="18" y="20"/>
-    <xacro:big_shelf name="zb_r6_l1" x="25" y="12"/>
-    <xacro:big_shelf name="zb_r6_l2" x="25" y="20"/>
-    <xacro:big_shelf name="zb_r7_l1" x="32" y="12"/>
-    <xacro:big_shelf name="zb_r7_l2" x="32" y="20"/>
-    <xacro:big_shelf name="zb_r8_l1" x="39" y="12"/>
-    <xacro:big_shelf name="zb_r8_l2" x="39" y="20"/>
-    <xacro:big_shelf name="zb_r9_l1" x="46" y="12"/>
-    <xacro:big_shelf name="zb_r9_l2" x="46" y="20"/>
-    <xacro:big_shelf name="zb_r10_l1" x="53" y="12"/>
-    <xacro:big_shelf name="zb_r10_l2" x="53" y="20"/>
-    <!-- ============================================================ -->
-    <!-- ZONE C: MEDIUM-DENSITY (big shelves, 3m aisles)              -->
-    <!-- x=-55 to +55, 16 rows, center-to-center 7m in X             -->
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
Commit message: Warehouse with fallen obstacles
Signed-off-by: SteveMacenski <stevenmacenski@gmail.com>

File: opennav_benchmark_sim/worlds/benchmark_warehouse.sdf.xacro (robot description, xacro)
@@ -177,4 +177,31 @@
         <name>${name}</name>
         <pose>${x} ${y} ${z} 0 0 ${yaw}</pose>
+        <static>true</static>
+      </include>
+    </xacro:macro>
+    <!-- Overturned pallet (tipped on side, roll=90deg) -->
+    <xacro:macro name="overturned_pallet" params="name x y yaw">
+      <include>
+        <uri>pallet_box_mobile</uri>
+        <name>${name}</name>
+        <pose>${x} ${y} 0.55 1.5708 0 ${yaw}</pose>
+        <static>true</static>
+      </include>
+    </xacro:macro>
+    <!-- Person (Fuel "Casual female" model from OpenRobotics) -->
+    <xacro:macro name="person" params="name x y yaw">
+      <include>
+        <uri>https://fuel.gazebosim.org/1.0/OpenRobotics/models/Casual female</uri>
+        <name>${name}</name>
+        <pose>${x} ${y} 0 0 0 ${yaw}</pose>
+        <static>true</static>
+      </include>
+    </xacro:macro>
+    <!-- Forklift (Fuel model from OpenRobotics) -->
+    <xacro:macro name="forklift" params="name x y yaw">
+      <include>
+        <uri>https://fuel.gazebosim.org/1.0/OpenRobotics/models/Forklift</uri>
+        <name>${name}</name>
+        <pose>${x} ${y} 0 0 0 ${yaw}</pose>
         <static>true</static>
       </include>
@@ -1607,4 +1634,18 @@
     <xacro:pallet name="ps_dock_13_9_L2" x="58.31" y="-53.93" z="1.21" yaw="-0.0048"/>
     <!-- Block-stack pallets: 718 models -->
+    <!-- ============================================================ -->
+    <!-- AISLE OBSTACLES (overturned pallets + people in Zone A)        -->
+    <!-- ============================================================ -->
+    <!-- Aisle 1: overturned pallets blocking aisle + 3 people -->
+    <xacro:overturned_pallet name="spill1_a" x="28.0" y="-34.4" yaw="0.3"/>
+    <xacro:overturned_pallet name="spill1_b" x="29.8" y="-34.25" yaw="-0.5"/>
+    <xacro:person name="spill1_p1" x="28.3" y="-33.6" yaw="-1.57"/>
+    <xacro:person name="spill1_p2" x="31.5" y="-34.199999999999996" yaw="3.14"/>
+    <xacro:person name="spill1_p3" x="28.9" y="-35.3" yaw="1.57"/>
+    <!-- Aisle 2: overturned pallets + person and forklift -->
+    <xacro:overturned_pallet name="spill2_a" x="-28.0" y="-14.8" yaw="-0.2"/>
+    <xacro:overturned_pallet name="spill2_b" x="-26.4" y="-14.9" yaw="0.45"/>
+    <xacro:forklift name="spill2_forklift" x="-25.6955" y="-10.5044" yaw="3.0"/>
+    <xacro:person name="spill2_p1" x="-24.5" y="-14.200000000000001" yaw="3.14"/>
   </world>
 </sdf>
