Commit message: simplified simulation for ~70% realtime on consumer weaker hardware
Signed-off-by: Steve Macenski <stevenmacenski@gmail.com>

File: opennav_benchmark_sim/worlds/benchmark_warehouse_simplified.sdf.xacro (robot description, xacro)
@@ -356,1359 +356,807 @@
     <xacro:support_column name="int_42" x="42.0" y="15"/>
     <!-- ============================================================ -->
-    <!-- ZONE A: BULK STORAGE (big shelves, back-to-back pairs, 2.0 m aisles) -->
-    <!-- 14 rows x 14 per row, aisle ~2.0m -->
+    <!-- SHELF VOLUMES - DERIVED FROM application/maps/benchmark_warehouse -->
+    <!-- 36 boxes extracted from the map's connected components, NOT the  -->
+    <!-- original per-shelf xacro positions: the original mesh's long axis -->
+    <!-- is in Y for big_shelf and yields one continuous 2.2 m x 72.5 m N-S -->
+    <!-- wall per shelf x-position. Box footprints, orientations, and gaps -->
+    <!-- now match the map exactly.                                       -->
+    <!--   14 big N-S vertical walls (zones A + B-west)                   -->
+    <!--    4 big E-W horizontal walls (zone D)                           -->
+    <!--   18 small E-W row-segments (zone B-east: 6, zone C: 12 with     -->
+    <!--      cross-aisle split)                                          -->
     <!-- ============================================================ -->
-    <xacro:big_shelf name="zone_a_r1_1" x="-54.0" y="-37.2"/>
-    <xacro:big_shelf name="zone_a_r1_2" x="-46.0" y="-37.2"/>
-    <xacro:big_shelf name="zone_a_r1_3" x="-38.0" y="-37.2"/>
-    <xacro:big_shelf name="zone_a_r1_4" x="-30.0" y="-37.2"/>
-    <xacro:big_shelf name="zone_a_r1_5" x="-22.0" y="-37.2"/>
-    <xacro:big_shelf name="zone_a_r1_6" x="-14.0" y="-37.2"/>
-    <xacro:big_shelf name="zone_a_r1_7" x="-6.0" y="-37.2"/>
-    <xacro:big_shelf name="zone_a_r1_8" x="10.0" y="-37.2"/>
-    <xacro:big_shelf name="zone_a_r1_9" x="18.0" y="-37.2"/>
-    <xacro:big_shelf name="zone_a_r1_10" x="26.0" y="-37.2"/>
-    <xacro:big_shelf name="zone_a_r1_11" x="34.0" y="-37.2"/>
-    <xacro:big_shelf name="zone_a_r1_12" x="42.0" y="-37.2"/>
-    <xacro:big_shelf name="zone_a_r1_13" x="50.0" y="-37.2"/>
-    <xacro:big_shelf name="zone_a_r1_14" x="58.0" y="-37.2"/>
-    <xacro:big_shelf name="zone_a_r2_1" x="-54.0" y="-36.0"/>
-    <xacro:big_shelf name="zone_a_r2_2" x="-46.0" y="-36.0"/>
-    <xacro:big_shelf name="zone_a_r2_3" x="-38.0" y="-36.0"/>
-    <xacro:big_shelf name="zone_a_r2_4" x="-30.0" y="-36.0"/>
-    <xacro:big_shelf name="zone_a_r2_5" x="-22.0" y="-36.0"/>
-    <xacro:big_shelf name="zone_a_r2_6" x="-14.0" y="-36.0"/>
-    <xacro:big_shelf name="zone_a_r2_7" x="-6.0" y="-36.0"/>
-    <xacro:big_shelf name="zone_a_r2_8" x="10.0" y="-36.0"/>
-    <xacro:big_shelf name="zone_a_r2_9" x="18.0" y="-36.0"/>
-    <xacro:big_shelf name="zone_a_r2_10" x="26.0" y="-36.0"/>
-    <xacro:big_shelf name="zone_a_r2_11" x="34.0" y="-36.0"/>
-    <xacro:big_shelf name="zone_a_r2_12" x="42.0" y="-36.0"/>
-    <xacro:big_shelf name="zone_a_r2_13" x="50.0" y="-36.0"/>
-    <xacro:big_shelf name="zone_a_r2_14" x="58.0" y="-36.0"/>
-    <xacro:big_shelf name="zone_a_r3_1" x="-54.0" y="-32.8"/>
-    <xacro:big_shelf name="zone_a_r3_2" x="-46.0" y="-32.8"/>
-    <xacro:big_shelf name="zone_a_r3_3" x="-38.0" y="-32.8"/>
-    <xacro:big_shelf name="zone_a_r3_4" x="-30.0" y="-32.8"/>
-    <xacro:big_shelf name="zone_a_r3_5" x="-22.0" y="-32.8"/>
-    <xacro:big_shelf name="zone_a_r3_6" x="-14.0" y="-32.8"/>
-    <xacro:big_shelf name="zone_a_r3_7" x="-6.0" y="-32.8"/>
-    <xacro:big_shelf name="zone_a_r3_8" x="10.0" y="-32.8"/>
-    <xacro:big_shelf name="zone_a_r3_9" x="18.0" y="-32.8"/>
-    <xacro:big_shelf name="zone_a_r3_10" x="26.0" y="-32.8"/>
-    <xacro:big_shelf name="zone_a_r3_11" x="34.0" y="-32.8"/>
-    <xacro:big_shelf name="zone_a_r3_12" x="42.0" y="-32.8"/>
-    <xacro:big_shelf name="zone_a_r3_13" x="50.0" y="-32.8"/>
-    <xacro:big_shelf name="zone_a_r3_14" x="58.0" y="-32.8"/>
-    <xacro:big_shelf name="zone_a_r4_1" x="-54.0" y="-31.6"/>
-    <xacro:big_shelf name="zone_a_r4_2" x="-46.0" y="-31.6"/>
-    <xacro:big_shelf name="zone_a_r4_3" x="-38.0" y="-31.6"/>
-    <xacro:big_shelf name="zone_a_r4_4" x="-30.0" y="-31.6"/>
-    <xacro:big_shelf name="zone_a_r4_5" x="-22.0" y="-31.6"/>
-    <xacro:big_shelf name="zone_a_r4_6" x="-14.0" y="-31.6"/>
-    <xacro:big_shelf name="zone_a_r4_7" x="-6.0" y="-31.6"/>
-    <xacro:big_shelf name="zone_a_r4_8" x="10.0" y="-31.6"/>
-    <xacro:big_shelf name="zone_a_r4_9" x="18.0" y="-31.6"/>
-    <xacro:big_shelf name="zone_a_r4_10" x="26.0" y="-31.6"/>
-    <xacro:big_shelf name="zone_a_r4_11" x="34.0" y="-31.6"/>
-    <xacro:big_shelf name="zone_a_r4_12" x="42.0" y="-31.6"/>
-    <xacro:big_shelf name="zone_a_r4_13" x="50.0" y="-31.6"/>
-    <xacro:big_shelf name="zone_a_r4_14" x="58.0" y="-31.6"/>
-    <xacro:big_shelf name="zone_a_r5_1" x="-54.0" y="-28.4"/>
-    <xacro:big_shelf name="zone_a_r5_2" x="-46.0" y="-28.4"/>
-    <xacro:big_shelf name="zone_a_r5_3" x="-38.0" y="-28.4"/>
-    <xacro:big_shelf name="zone_a_r5_4" x="-30.0" y="-28.4"/>
-    <xacro:big_shelf name="zone_a_r5_5" x="-22.0" y="-28.4"/>
-    <xacro:big_shelf name="zone_a_r5_6" x="-14.0" y="-28.4"/>
-    <xacro:big_shelf name="zone_a_r5_7" x="-6.0" y="-28.4"/>
-    <xacro:big_shelf name="zone_a_r5_8" x="10.0" y="-28.4"/>
-    <xacro:big_shelf name="zone_a_r5_9" x="18.0" y="-28.4"/>
-    <xacro:big_shelf name="zone_a_r5_10" x="26.0" y="-28.4"/>
-    <xacro:big_shelf name="zone_a_r5_11" x="34.0" y="-28.4"/>
-    <xacro:big_shelf name="zone_a_r5_12" x="42.0" y="-28.4"/>
-    <xacro:big_shelf name="zone_a_r5_13" x="50.0" y="-28.4"/>
-    <xacro:big_shelf name="zone_a_r5_14" x="58.0" y="-28.4"/>
-    <xacro:big_shelf name="zone_a_r6_1" x="-54.0" y="-27.2"/>
-    <xacro:big_shelf name="zone_a_r6_2" x="-46.0" y="-27.2"/>
-    <xacro:big_shelf name="zone_a_r6_3" x="-38.0" y="-27.2"/>
-    <xacro:big_shelf name="zone_a_r6_4" x="-30.0" y="-27.2"/>
-    <xacro:big_shelf name="zone_a_r6_5" x="-22.0" y="-27.2"/>
-    <xacro:big_shelf name="zone_a_r6_6" x="-14.0" y="-27.2"/>
-    <xacro:big_shelf name="zone_a_r6_7" x="-6.0" y="-27.2"/>
-    <xacro:big_shelf name="zone_a_r6_8" x="10.0" y="-27.2"/>
-    <xacro:big_shelf name="zone_a_r6_9" x="18.0" y="-27.2"/>
-    <xacro:big_shelf name="zone_a_r6_10" x="26.0" y="-27.2"/>
-    <xacro:big_shelf name="zone_a_r6_11" x="34.0" y="-27.2"/>
-    <xacro:big_shelf name="zone_a_r6_12" x="42.0" y="-27.2"/>
-    <xacro:big_shelf name="zone_a_r6_13" x="50.0" y="-27.2"/>
-    <xacro:big_shelf name="zone_a_r6_14" x="58.0" y="-27.2"/>
-    <xacro:big_shelf name="zone_a_r7_1" x="-54.0" y="-22.0"/>
-    <xacro:big_shelf name="zone_a_r7_2" x="-46.0" y="-22.0"/>
-    <xacro:big_shelf name="zone_a_r7_3" x="-38.0" y="-22.0"/>
-    <xacro:big_shelf name="zone_a_r7_4" x="-30.0" y="-22.0"/>
-    <xacro:big_shelf name="zone_a_r7_5" x="-22.0" y="-22.0"/>
-    <xacro:big_shelf name="zone_a_r7_6" x="-14.0" y="-22.0"/>
-    <xacro:big_shelf name="zone_a_r7_7" x="-6.0" y="-22.0"/>
-    <xacro:big_shelf name="zone_a_r7_8" x="10.0" y="-22.0"/>
-    <xacro:big_shelf name="zone_a_r7_9" x="18.0" y="-22.0"/>
-    <xacro:big_shelf name="zone_a_r7_10" x="26.0" y="-22.0"/>
-    <xacro:big_shelf name="zone_a_r7_11" x="34.0" y="-22.0"/>
-    <xacro:big_shelf name="zone_a_r7_12" x="42.0" y="-22.0"/>
-    <xacro:big_shelf name="zone_a_r7_13" x="50.0" y="-22.0"/>
-    <xacro:big_shelf name="zone_a_r7_14" x="58.0" y="-22.0"/>
-    <xacro:big_shelf name="zone_a_r8_1" x="-54.0" y="-20.8"/>
-    <xacro:big_shelf name="zone_a_r8_2" x="-46.0" y="-20.8"/>
-    <xacro:big_shelf name="zone_a_r8_3" x="-38.0" y="-20.8"/>
-    <xacro:big_shelf name="zone_a_r8_4" x="-30.0" y="-20.8"/>
-    <xacro:big_shelf name="zone_a_r8_5" x="-22.0" y="-20.8"/>
-    <xacro:big_shelf name="zone_a_r8_6" x="-14.0" y="-20.8"/>
-    <xacro:big_shelf name="zone_a_r8_7" x="-6.0" y="-20.8"/>
-    <xacro:big_shelf name="zone_a_r8_8" x="10.0" y="-20.8"/>
-    <xacro:big_shelf name="zone_a_r8_9" x="18.0" y="-20.8"/>
-    <xacro:big_shelf name="zone_a_r8_10" x="26.0" y="-20.8"/>
-    <xacro:big_shelf name="zone_a_r8_11" x="34.0" y="-20.8"/>
-    <xacro:big_shelf name="zone_a_r8_12" x="42.0" y="-20.8"/>
-    <xacro:big_shelf name="zone_a_r8_13" x="50.0" y="-20.8"/>
-    <xacro:big_shelf name="zone_a_r8_14" x="58.0" y="-20.8"/>
-    <xacro:big_shelf name="zone_a_r9_1" x="-54.0" y="-17.6"/>
-    <xacro:big_shelf name="zone_a_r9_2" x="-46.0" y="-17.6"/>
-    <xacro:big_shelf name="zone_a_r9_3" x="-38.0" y="-17.6"/>
-    <xacro:big_shelf name="zone_a_r9_4" x="-30.0" y="-17.6"/>
-    <xacro:big_shelf name="zone_a_r9_5" x="-22.0" y="-17.6"/>
-    <xacro:big_shelf name="zone_a_r9_6" x="-14.0" y="-17.6"/>
-    <xacro:big_shelf name="zone_a_r9_7" x="-6.0" y="-17.6"/>
-    <xacro:big_shelf name="zone_a_r9_8" x="10.0" y="-17.6"/>
-    <xacro:big_shelf name="zone_a_r9_9" x="18.0" y="-17.6"/>
-    <xacro:big_shelf name="zone_a_r9_10" x="26.0" y="-17.6"/>
-    <xacro:big_shelf name="zone_a_r9_11" x="34.0" y="-17.6"/>
-    <xacro:big_shelf name="zone_a_r9_12" x="42.0" y="-17.6"/>
-    <xacro:big_shelf name="zone_a_r9_13" x="50.0" y="-17.6"/>
-    <xacro:big_shelf name="zone_a_r9_14" x="58.0" y="-17.6"/>
-    <xacro:big_shelf name="zone_a_r10_1" x="-54.0" y="-16.4"/>
-    <xacro:big_shelf name="zone_a_r10_2" x="-46.0" y="-16.4"/>
-    <xacro:big_shelf name="zone_a_r10_3" x="-38.0" y="-16.4"/>
-    <xacro:big_shelf name="zone_a_r10_4" x="-30.0" y="-16.4"/>
-    <xacro:big_shelf name="zone_a_r10_5" x="-22.0" y="-16.4"/>
-    <xacro:big_shelf name="zone_a_r10_6" x="-14.0" y="-16.4"/>
-    <xacro:big_shelf name="zone_a_r10_7" x="-6.0" y="-16.4"/>
-    <xacro:big_shelf name="zone_a_r10_8" x="10.0" y="-16.4"/>
-    <xacro:big_shelf name="zone_a_r10_9" x="18.0" y="-16.4"/>
-    <xacro:big_shelf name="zone_a_r10_10" x="26.0" y="-16.4"/>
-    <xacro:big_shelf name="zone_a_r10_11" x="34.0" y="-16.4"/>
-    <xacro:big_shelf name="zone_a_r10_12" x="42.0" y="-16.4"/>
-    <xacro:big_shelf name="zone_a_r10_13" x="50.0" y="-16.4"/>
-    <xacro:big_shelf name="zone_a_r10_14" x="58.0" y="-16.4"/>
-    <xacro:big_shelf name="zone_a_r11_1" x="-54.0" y="-13.2"/>
-    <xacro:big_shelf name="zone_a_r11_2" x="-46.0" y="-13.2"/>
-    <xacro:big_shelf name="zone_a_r11_3" x="-38.0" y="-13.2"/>
-    <xacro:big_shelf name="zone_a_r11_4" x="-30.0" y="-13.2"/>
-    <xacro:big_shelf name="zone_a_r11_5" x="-22.0" y="-13.2"/>
-    <xacro:big_shelf name="zone_a_r11_6" x="-14.0" y="-13.2"/>
-    <xacro:big_shelf name="zone_a_r11_7" x="-6.0" y="-13.2"/>
-    <xacro:big_shelf name="zone_a_r11_8" x="10.0" y="-13.2"/>
-    <xacro:big_shelf name="zone_a_r11_9" x="18.0" y="-13.2"/>
-    <xacro:big_shelf name="zone_a_r11_10" x="26.0" y="-13.2"/>
-    <xacro:big_shelf name="zone_a_r11_11" x="34.0" y="-13.2"/>
-    <xacro:big_shelf name="zone_a_r11_12" x="42.0" y="-13.2"/>
-    <xacro:big_shelf name="zone_a_r11_13" x="50.0" y="-13.2"/>
-    <xacro:big_shelf name="zone_a_r11_14" x="58.0" y="-13.2"/>
-    <xacro:big_shelf name="zone_a_r12_1" x="-54.0" y="-12.0"/>
-    <xacro:big_shelf name="zone_a_r12_2" x="-46.0" y="-12.0"/>
-    <xacro:big_shelf name="zone_a_r12_3" x="-38.0" y="-12.0"/>
-    <xacro:big_shelf name="zone_a_r12_4" x="-30.0" y="-12.0"/>
-    <xacro:big_shelf name="zone_a_r12_5" x="-22.0" y="-12.0"/>
-    <xacro:big_shelf name="zone_a_r12_6" x="-14.0" y="-12.0"/>
-    <xacro:big_shelf name="zone_a_r12_7" x="-6.0" y="-12.0"/>
-    <xacro:big_shelf name="zone_a_r12_8" x="10.0" y="-12.0"/>
-    <xacro:big_shelf name="zone_a_r12_9" x="18.0" y="-12.0"/>
-    <xacro:big_shelf name="zone_a_r12_10" x="26.0" y="-12.0"/>
-    <xacro:big_shelf name="zone_a_r12_11" x="34.0" y="-12.0"/>
-    <xacro:big_shelf name="zone_a_r12_12" x="42.0" y="-12.0"/>
-    <xacro:big_shelf name="zone_a_r12_13" x="50.0" y="-12.0"/>
-    <xacro:big_shelf name="zone_a_r12_14" x="58.0" y="-12.0"/>
-    <xacro:big_shelf name="zone_a_r13_1" x="-54.0" y="-8.8"/>
-    <xacro:big_shelf name="zone_a_r13_2" x="-46.0" y="-8.8"/>
-    <xacro:big_shelf name="zone_a_r13_3" x="-38.0" y="-8.8"/>
-    <xacro:big_shelf name="zone_a_r13_4" x="-30.0" y="-8.8"/>
-    <xacro:big_shelf name="zone_a_r13_5" x="-22.0" y="-8.8"/>
-    <xacro:big_shelf name="zone_a_r13_6" x="-14.0" y="-8.8"/>
-    <xacro:big_shelf name="zone_a_r13_7" x="-6.0" y="-8.8"/>
-    <xacro:big_shelf name="zone_a_r13_8" x="10.0" y="-8.8"/>
-    <xacro:big_shelf name="zone_a_r13_9" x="18.0" y="-8.8"/>
-    <xacro:big_shelf name="zone_a_r13_10" x="26.0" y="-8.8"/>
-    <xacro:big_shelf name="zone_a_r13_11" x="34.0" y="-8.8"/>
-    <xacro:big_shelf name="zone_a_r13_12" x="42.0" y="-8.8"/>
-    <xacro:big_shelf name="zone_a_r13_13" x="50.0" y="-8.8"/>
-    <xacro:big_shelf name="zone_a_r13_14" x="58.0" y="-8.8"/>
-    <xacro:big_shelf name="zone_a_r14_1" x="-54.0" y="-7.6"/>
-    <xacro:big_shelf name="zone_a_r14_2" x="-46.0" y="-7.6"/>
-    <xacro:big_shelf name="zone_a_r14_3" x="-38.0" y="-7.6"/>
-    <xacro:big_shelf name="zone_a_r14_4" x="-30.0" y="-7.6"/>
-    <xacro:big_shelf name="zone_a_r14_5" x="-22.0" y="-7.6"/>
-    <xacro:big_shelf name="zone_a_r14_6" x="-14.0" y="-7.6"/>
-    <xacro:big_shelf name="zone_a_r14_7" x="-6.0" y="-7.6"/>
-    <xacro:big_shelf name="zone_a_r14_8" x="10.0" y="-7.6"/>
-    <xacro:big_shelf name="zone_a_r14_9" x="18.0" y="-7.6"/>
-    <xacro:big_shelf name="zone_a_r14_10" x="26.0" y="-7.6"/>
-    <xacro:big_shelf name="zone_a_r14_11" x="34.0" y="-7.6"/>
-    <xacro:big_shelf name="zone_a_r14_12" x="42.0" y="-7.6"/>
-    <xacro:big_shelf name="zone_a_r14_13" x="50.0" y="-7.6"/>
-    <xacro:big_shelf name="zone_a_r14_14" x="58.0" y="-7.6"/>
-    <!-- zone_a shelves (big): 196 -->
+    <!-- Big N-S vertical shelves (zones A + B-west: 14 walls @ ~2.2m x 72.5m / 47.7m x 6m) -->
+    <model name="shelf_ns_01">
+      <static>true</static>
+      <pose>-54.525 -10.025 3.000 0 0 0</pose>
+      <link name="link">
+        <visual name="visual">
+          <geometry><box><size>2.200 72.500 6.000</size></box></geometry>
+          <material>
+            <ambient>0.40 0.30 0.18 1</ambient>
+            <diffuse>0.40 0.30 0.18 1</diffuse>
+            <specular>0.1 0.1 0.1 1</specular>
+          </material>
+        </visual>
+        <collision name="collision">
+          <geometry><box><size>2.200 72.500 6.000</size></box></geometry>
+        </collision>
+      </link>
+    </model>
+    <model name="shelf_ns_02">
+      <static>true</static>
+      <pose>-46.525 -10.025 3.000 0 0 0</pose>
+      <link name="link">
+        <visual name="visual">
+          <geometry><box><size>2.200 72.500 6.000</size></box></geometry>
+          <material>
+            <ambient>0.40 0.30 0.18 1</ambient>
+            <diffuse>0.40 0.30 0.18 1</diffuse>
+            <specular>0.1 0.1 0.1 1</specular>
+          </material>
+        </visual>
+        <collision name="collision">
+          <geometry><box><size>2.200 72.500 6.000</size></box></geometry>
+        </collision>
+      </link>
+    </model>
+    <model name="shelf_ns_03">
+      <static>true</static>
+      <pose>-38.525 -10.025 3.000 0 0 0</pose>
+      <link name="link">
+        <visual name="visual">
+          <geometry><box><size>2.200 72.500 6.000</size></box></geometry>
+          <material>
+            <ambient>0.40 0.30 0.18 1</ambient>
+            <diffuse>0.40 0.30 0.18 1</diffuse>
+            <specular>0.1 0.1 0.1 1</specular>
+          </material>
+        </visual>
+        <collision name="collision">
+          <geometry><box><size>2.200 72.500 6.000</size></box></geometry>
+        </collision>
+      </link>
+    </model>
+    <model name="shelf_ns_04">
+      <static>true</static>
+      <pose>-30.525 -10.025 3.000 0 0 0</pose>
+      <link name="link">
+        <visual name="visual">
+          <geometry><box><size>2.200 72.500 6.000</size></box></geometry>
+          <material>
+            <ambient>0.40 0.30 0.18 1</ambient>
+            <diffuse>0.40 0.30 0.18 1</diffuse>
+            <specular>0.1 0.1 0.1 1</specular>
+          </material>
+        </visual>
+        <collision name="collision">
+          <geometry><box><size>2.200 72.500 6.000</size></box></geometry>
+        </collision>
+      </link>
+    </model>
+    <model name="shelf_ns_05">
+      <static>true</static>
+      <pose>-22.525 -10.025 3.000 0 0 0</pose>
+      <link name="link">
+        <visual name="visual">
+          <geometry><box><size>2.200 72.500 6.000</size></box></geometry>
+          <material>
+            <ambient>0.40 0.30 0.18 1</ambient>
+            <diffuse>0.40 0.30 0.18 1</diffuse>
+            <specular>0.1 0.1 0.1 1</specular>
+          </material>
+        </visual>
+        <collision name="collision">
+          <geometry><box><size>2.200 72.500 6.000</size></box></geometry>
+        </collision>
+      </link>
+    </model>
+    <model name="shelf_ns_06">
+      <static>true</static>
+      <pose>-14.525 -10.025 3.000 0 0 0</pose>
+      <link name="link">
+        <visual name="visual">
+          <geometry><box><size>2.200 72.500 6.000</size></box></geometry>
+          <material>
+            <ambient>0.40 0.30 0.18 1</ambient>
+            <diffuse>0.40 0.30 0.18 1</diffuse>
+            <specular>0.1 0.1 0.1 1</specular>
+          </material>
+        </visual>
+        <collision name="collision">
+          <geometry><box><size>2.200 72.500 6.000</size></box></geometry>
+        </collision>
+      </link>
+    </model>
+    <model name="shelf_ns_07">
+      <static>true</static>
+      <pose>-6.525 -10.025 3.000 0 0 0</pose>
+      <link name="link">
+        <visual name="visual">
+          <geometry><box><size>2.200 72.500 6.000</size></box></geometry>
+          <material>
+            <ambient>0.40 0.30 0.18 1</ambient>
+            <diffuse>0.40 0.30 0.18 1</diffuse>
+            <specular>0.1 0.1 0.1 1</specular>
+          </material>
+        </visual>
+        <collision name="collision">
+          <geometry><box><size>2.200 72.500 6.000</size></box></geometry>
+        </collision>
+      </link>
+    </model>
+    <model name="shelf_ns_08">
+      <static>true</static>
+      <pose>9.475 -22.425 3.000 0 0 0</pose>
+      <link name="link">
+        <visual name="visual">
+          <geometry><box><size>2.200 47.700 6.000</size></box></geometry>
+          <material>
+            <ambient>0.40 0.30 0.18 1</ambient>
+            <diffuse>0.40 0.30 0.18 1</diffuse>
+            <specular>0.1 0.1 0.1 1</specular>
+          </material>
+        </visual>
+        <collision name="collision">
+          <geometry><box><size>2.200 47.700 6.000</size></box></geometry>
+        </collision>
+      </link>
+    </model>
+    <model name="shelf_ns_09">
+      <static>true</static>
+      <pose>17.475 -22.425 3.000 0 0 0</pose>
+      <link name="link">
+        <visual name="visual">
+          <geometry><box><size>2.200 47.700 6.000</size></box></geometry>
+          <material>
+            <ambient>0.40 0.30 0.18 1</ambient>
+            <diffuse>0.40 0.30 0.18 1</diffuse>
+            <specular>0.1 0.1 0.1 1</specular>
+          </material>
+        </visual>
+        <collision name="collision">
+          <geometry><box><size>2.200 47.700 6.000</size></box></geometry>
+        </collision>
+      </link>
+    </model>
+    <model name="shelf_ns_10">
+      <static>true</static>
+      <pose>25.475 -22.425 3.000 0 0 0</pose>
+      <link name="link">
+        <visual name="visual">
+          <geometry><box><size>2.200 47.700 6.000</size></box></geometry>
+          <material>
+            <ambient>0.40 0.30 0.18 1</ambient>
+            <diffuse>0.40 0.30 0.18 1</diffuse>
+            <specular>0.1 0.1 0.1 1</specular>
+          </material>
+        </visual>
+        <collision name="collision">
+          <geometry><box><size>2.200 47.700 6.000</size></box></geometry>
+        </collision>
+      </link>
+    </model>
+    <model name="shelf_ns_11">
+      <static>true</static>
+      <pose>33.475 -22.425 3.000 0 0 0</pose>
+      <link name="link">
+        <visual name="visual">
+          <geometry><box><size>2.200 47.700 6.000</size></box></geometry>
+          <material>
+            <ambient>0.40 0.30 0.18 1</ambient>
+            <diffuse>0.40 0.30 0.18 1</diffuse>
+            <specular>0.1 0.1 0.1 1</specular>
+          </material>
+        </visual>
+        <collision name="collision">
+          <geometry><box><size>2.200 47.700 6.000</size></box></geometry>
+        </collision>
+      </link>
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