Commit message: more incremental simulation improvements
Signed-off-by: SteveMacenski <stevenmacenski@gmail.com>

File: opennav_benchmark_robot/urdf/benchmark_robot.sdf.xacro (robot description, xacro)
@@ -44,7 +44,7 @@
       <child>base_link</child>
     </joint>
-    <!-- ============ SENSOR TOWER (front, Nav2 grey) ============ -->
+    <!-- ============ SENSOR TOWER (front arc panel, Nav2 blue) ============ -->
     <link name="sensor_tower_link">
-      <pose relative_to="base_link">0.15 0 0.31 0 0 0</pose>
+      <pose relative_to="base_link">0.52 0 0.318 0 0 0</pose>
       <inertial>
         <mass>3.0</mass>
@@ -61,7 +61,7 @@
         </geometry>
         <material>
-          <ambient>0.6 0.62 0.65 1.0</ambient>
-          <diffuse>0.6 0.62 0.65 1.0</diffuse>
-          <specular>0.05 0.05 0.05 1.0</specular>
+          <ambient>0.28 0.66 0.85 1.0</ambient>
+          <diffuse>0.28 0.66 0.85 1.0</diffuse>
+          <specular>0.1 0.1 0.1 1.0</specular>
         </material>
       </visual>
@@ -225,5 +225,5 @@
     <!-- Center: top of tower, 360deg, 32ch, 75m -->
     <link name="lidar_3d_center_link">
-      <pose relative_to="sensor_tower_link">0 0 0.17 0 0 0</pose>
+      <pose relative_to="sensor_tower_link">0 0 0.167 0 0 0</pose>
       <inertial>
         <mass>0.5</mass>
@@ -289,5 +289,5 @@
     <!-- Front-left: on left arm, 120deg, 16ch, 30m, tilted down 15deg -->
     <link name="lidar_3d_front_left_link">
-      <pose relative_to="sensor_tower_link">0 0.24 0.17 -0.2618 0 0</pose>
+      <pose relative_to="sensor_tower_link">0 0.24 0.148 -0.2618 0 0</pose>
       <inertial>
         <mass>0.5</mass>
@@ -353,5 +353,5 @@
     <!-- Front-right: on right arm, 120deg, 16ch, 30m, tilted down 15deg -->
     <link name="lidar_3d_front_right_link">
-      <pose relative_to="sensor_tower_link">0 -0.24 0.17 0.2618 0 0</pose>
+      <pose relative_to="sensor_tower_link">0 -0.24 0.148 0.2618 0 0</pose>
       <inertial>
         <mass>0.5</mass>

File: opennav_benchmark_robot/urdf/benchmark_robot.urdf.xacro (robot description, xacro)
@@ -13,7 +13,7 @@
   <xacro:property name="caster_radius" value="0.05"/>
   <xacro:property name="caster_mass" value="0.5"/>
-  <!-- Tower: sits on chassis top at front area -->
-  <xacro:property name="tower_x" value="0.15"/>
-  <xacro:property name="tower_half_h" value="0.15"/>
+  <!-- Tower: arc panel at front, bottom aligns with chassis top -->
+  <xacro:property name="tower_x" value="0.52"/>
+  <xacro:property name="tower_z_offset" value="0.318"/>
   <!-- Colors -->
   <material name="nav2_blue">
@@ -84,5 +84,5 @@
         <mesh filename="package://opennav_benchmark_robot/meshes/sensor_tower.stl"/>
       </geometry>
-      <material name="nav2_grey"/>
+      <material name="nav2_blue"/>
     </visual>
     <inertial>
@@ -94,5 +94,5 @@
     <parent link="base_link"/>
     <child link="sensor_tower_link"/>
-    <origin xyz="${tower_x} 0 ${chassis_height/2 + tower_half_h}" rpy="0 0 0"/>
+    <origin xyz="${tower_x} 0 ${tower_z_offset}" rpy="0 0 0"/>
   </joint>
   <!-- ============ DRIVE WHEELS ============ -->
@@ -181,5 +181,5 @@
     <parent link="sensor_tower_link"/>
     <child link="lidar_3d_center_link"/>
-    <origin xyz="0 0 ${tower_half_h + 0.01}" rpy="0 0 0"/>
+    <origin xyz="0 0 0.167" rpy="0 0 0"/>
   </joint>
   <!-- Front-left: on left arm of tower crossbar -->
@@ -202,5 +202,5 @@
     <parent link="sensor_tower_link"/>
     <child link="lidar_3d_front_left_link"/>
-    <origin xyz="0 0.22 ${tower_half_h + 0.02}" rpy="${-pi/12} 0 0"/>
+    <origin xyz="0 0.24 0.148" rpy="${-pi/12} 0 0"/>
   </joint>
   <!-- Front-right: on right arm of tower crossbar -->
@@ -223,5 +223,5 @@
     <parent link="sensor_tower_link"/>
     <child link="lidar_3d_front_right_link"/>
-    <origin xyz="0 -0.22 ${tower_half_h + 0.02}" rpy="${pi/12} 0 0"/>
+    <origin xyz="0 -0.24 0.148" rpy="${pi/12} 0 0"/>
   </joint>
   <!-- ============ 2D LIDARS (SICK TiM781 on chassis corners) ============ -->

Commit message: forklift chassis now
Signed-off-by: SteveMacenski <stevenmacenski@gmail.com>

File: opennav_benchmark_robot/urdf/benchmark_robot.sdf.xacro (robot description, xacro)
@@ -25,12 +25,8 @@
       <visual name="chassis_visual">
         <visibility_flags>${robot_visibility_flags}</visibility_flags>
-        <geometry>
-          <mesh><uri>package://opennav_benchmark_robot/meshes/chassis_body.stl</uri></mesh>
-        </geometry>
-        <material>
-          <ambient>0.28 0.66 0.85 1.0</ambient>
-          <diffuse>0.28 0.66 0.85 1.0</diffuse>
-          <specular>0.1 0.1 0.1 1.0</specular>
-        </material>
+        <pose>0 0 -0.25 1.5708 0 -1.5708</pose>
+        <geometry>
+          <mesh><uri>package://opennav_benchmark_robot/meshes/Forklift_agv_01.obj</uri></mesh>
+        </geometry>
       </visual>
       <collision name="chassis_collision">
@@ -43,31 +39,4 @@
       <parent>base_footprint</parent>
       <child>base_link</child>
-    </joint>
-    <!-- ============ SENSOR TOWER (front arc panel, Nav2 blue) ============ -->
-    <link name="sensor_tower_link">
-      <pose relative_to="base_link">0.52 0 0.318 0 0 0</pose>
-      <inertial>
-        <mass>3.0</mass>
-        <inertia>
-          <ixx>0.03</ixx><ixy>0</ixy><ixz>0</ixz>
-          <iyy>0.03</iyy><iyz>0</iyz>
-          <izz>0.01</izz>
-        </inertia>
-      </inertial>
-      <visual name="tower_visual">
-        <visibility_flags>${robot_visibility_flags}</visibility_flags>
-        <geometry>
-          <mesh><uri>package://opennav_benchmark_robot/meshes/sensor_tower.stl</uri></mesh>
-        </geometry>
-        <material>
-          <ambient>0.28 0.66 0.85 1.0</ambient>
-          <diffuse>0.28 0.66 0.85 1.0</diffuse>
-          <specular>0.1 0.1 0.1 1.0</specular>
-        </material>
-      </visual>
-    </link>
-    <joint name="sensor_tower_joint" type="fixed">
-      <parent>base_link</parent>
-      <child>sensor_tower_link</child>
     </joint>
     <!-- ============ DRIVE WHEELS ============ -->
@@ -201,5 +170,5 @@
       <sensor name="imu_sensor" type="imu">
         <always_on>true</always_on>
-        <update_rate>200</update_rate>
+        <update_rate>100</update_rate>
         <imu>
           <angular_velocity>
@@ -244,9 +213,4 @@
         </material>
       </visual>
-      <collision name="collision">
-        <geometry>
-          <cylinder><radius>0.0425</radius><length>0.085</length></cylinder>
-        </geometry>
-      </collision>
       <sensor name="lidar_3d_center_sensor" type="gpu_lidar">
         <always_on>true</always_on>
@@ -269,5 +233,5 @@
           <range>
             <min>0.3</min>
-            <max>75.0</max>
+            <max>50.0</max>
             <resolution>0.01</resolution>
           </range>
@@ -308,9 +272,4 @@
         </material>
       </visual>
-      <collision name="collision">
-        <geometry>
-          <cylinder><radius>0.0425</radius><length>0.085</length></cylinder>
-        </geometry>
-      </collision>
       <sensor name="lidar_3d_front_left_sensor" type="gpu_lidar">
         <always_on>true</always_on>
@@ -372,9 +331,4 @@
         </material>
       </visual>
-      <collision name="collision">
-        <geometry>
-          <cylinder><radius>0.0425</radius><length>0.085</length></cylinder>
-        </geometry>
-      </collision>
       <sensor name="lidar_3d_front_right_sensor" type="gpu_lidar">
         <always_on>true</always_on>
@@ -436,12 +390,7 @@
         </material>
       </visual>
-      <collision name="collision">
-        <geometry>
-          <cylinder><radius>0.03</radius><length>0.095</length></cylinder>
-        </geometry>
-      </collision>
       <sensor name="lidar_2d_front_sensor" type="gpu_lidar">
         <always_on>true</always_on>
-        <update_rate>10</update_rate>
+        <update_rate>30</update_rate>
         <lidar>
           <scan>
@@ -499,12 +448,7 @@
         </material>
       </visual>
-      <collision name="collision">
-        <geometry>
-          <cylinder><radius>0.03</radius><length>0.095</length></cylinder>
-        </geometry>
-      </collision>
       <sensor name="lidar_2d_rear_sensor" type="gpu_lidar">
         <always_on>true</always_on>
-        <update_rate>10</update_rate>
+        <update_rate>30</update_rate>
         <lidar>
           <scan>
@@ -564,9 +508,4 @@
           </material>
         </visual>
-        <collision name="collision">
-          <geometry>
-            <box><size>0.025 0.09 0.025</size></box>
-          </geometry>
-        </collision>
         <sensor name="${name}_rgbd" type="rgbd_camera">
           <always_on>true</always_on>
@@ -580,5 +519,5 @@
             <clip>
               <near>0.1</near>
-              <far>10.0</far>
+              <far>7.0</far>
             </clip>
           </camera>

File: opennav_benchmark_robot/urdf/benchmark_robot.urdf.xacro (robot description, xacro)
@@ -61,8 +61,8 @@
   <link name="base_link">
     <visual>
-      <geometry>
-        <mesh filename="package://opennav_benchmark_robot/meshes/chassis_body.stl"/>
-      </geometry>
-      <material name="nav2_blue"/>
+      <origin xyz="0 0 -0.25" rpy="1.5708 0 -1.5708"/>
+      <geometry>
+        <mesh filename="package://opennav_benchmark_robot/meshes/Forklift_agv_01.obj"/>
+      </geometry>
     </visual>
     <collision>
@@ -80,10 +80,5 @@
   <!-- ============ SENSOR TOWER ============ -->
   <link name="sensor_tower_link">
-    <visual>
-      <geometry>
-        <mesh filename="package://opennav_benchmark_robot/meshes/sensor_tower.stl"/>
-      </geometry>
-      <material name="nav2_blue"/>
-    </visual>
+    <!-- sensor_tower visual removed (forklift mesh replaces it) -->
     <inertial>
       <mass value="3.0"/>
