Commit message: forklift chassis now
Signed-off-by: SteveMacenski <stevenmacenski@gmail.com>

File: opennav_benchmark_sim/worlds/benchmark_warehouse.sdf.xacro (robot description, xacro)
@@ -253,228 +253,264 @@
     <!-- ============================================================ -->
     <!-- ZONE A: BULK STORAGE (big shelves, back-to-back pairs, 2.0 m aisles) -->
-    <!-- 14 rows x 12 per row, aisle ~2.0m -->
-    <!-- ============================================================ -->
-    <xacro:big_shelf name="zone_a_r1_1" x="-54" y="-37.2"/>
-    <xacro:big_shelf name="zone_a_r1_2" x="-46.0" y="-37.2"/>
-    <xacro:big_shelf name="zone_a_r1_3" x="-38.0" y="-37.2"/>
-    <xacro:big_shelf name="zone_a_r1_4" x="-30.0" y="-37.2"/>
-    <xacro:big_shelf name="zone_a_r1_5" x="-22.0" y="-37.2"/>
-    <xacro:big_shelf name="zone_a_r1_6" x="-14.0" y="-37.2"/>
-    <xacro:big_shelf name="zone_a_r1_7" x="10.0" y="-37.2"/>
-    <xacro:big_shelf name="zone_a_r1_8" x="18.0" y="-37.2"/>
-    <xacro:big_shelf name="zone_a_r1_9" x="26.0" y="-37.2"/>
-    <xacro:big_shelf name="zone_a_r1_10" x="34.0" y="-37.2"/>
-    <xacro:big_shelf name="zone_a_r1_11" x="42.0" y="-37.2"/>
-    <xacro:big_shelf name="zone_a_r1_12" x="50.0" y="-37.2"/>
-    <xacro:big_shelf name="zone_a_r2_1" x="-54" y="-36.0"/>
-    <xacro:big_shelf name="zone_a_r2_2" x="-46.0" y="-36.0"/>
-    <xacro:big_shelf name="zone_a_r2_3" x="-38.0" y="-36.0"/>
-    <xacro:big_shelf name="zone_a_r2_4" x="-30.0" y="-36.0"/>
-    <xacro:big_shelf name="zone_a_r2_5" x="-22.0" y="-36.0"/>
-    <xacro:big_shelf name="zone_a_r2_6" x="-14.0" y="-36.0"/>
-    <xacro:big_shelf name="zone_a_r2_7" x="10.0" y="-36.0"/>
-    <xacro:big_shelf name="zone_a_r2_8" x="18.0" y="-36.0"/>
-    <xacro:big_shelf name="zone_a_r2_9" x="26.0" y="-36.0"/>
-    <xacro:big_shelf name="zone_a_r2_10" x="34.0" y="-36.0"/>
-    <xacro:big_shelf name="zone_a_r2_11" x="42.0" y="-36.0"/>
-    <xacro:big_shelf name="zone_a_r2_12" x="50.0" y="-36.0"/>
-    <xacro:big_shelf name="zone_a_r3_1" x="-54" y="-32.8"/>
-    <xacro:big_shelf name="zone_a_r3_2" x="-46.0" y="-32.8"/>
-    <xacro:big_shelf name="zone_a_r3_3" x="-38.0" y="-32.8"/>
-    <xacro:big_shelf name="zone_a_r3_4" x="-30.0" y="-32.8"/>
-    <xacro:big_shelf name="zone_a_r3_5" x="-22.0" y="-32.8"/>
-    <xacro:big_shelf name="zone_a_r3_6" x="-14.0" y="-32.8"/>
-    <xacro:big_shelf name="zone_a_r3_7" x="10.0" y="-32.8"/>
-    <xacro:big_shelf name="zone_a_r3_8" x="18.0" y="-32.8"/>
-    <xacro:big_shelf name="zone_a_r3_9" x="26.0" y="-32.8"/>
-    <xacro:big_shelf name="zone_a_r3_10" x="34.0" y="-32.8"/>
-    <xacro:big_shelf name="zone_a_r3_11" x="42.0" y="-32.8"/>
-    <xacro:big_shelf name="zone_a_r3_12" x="50.0" y="-32.8"/>
-    <xacro:big_shelf name="zone_a_r4_1" x="-54" y="-31.6"/>
-    <xacro:big_shelf name="zone_a_r4_2" x="-46.0" y="-31.6"/>
-    <xacro:big_shelf name="zone_a_r4_3" x="-38.0" y="-31.6"/>
-    <xacro:big_shelf name="zone_a_r4_4" x="-30.0" y="-31.6"/>
-    <xacro:big_shelf name="zone_a_r4_5" x="-22.0" y="-31.6"/>
-    <xacro:big_shelf name="zone_a_r4_6" x="-14.0" y="-31.6"/>
-    <xacro:big_shelf name="zone_a_r4_7" x="10.0" y="-31.6"/>
-    <xacro:big_shelf name="zone_a_r4_8" x="18.0" y="-31.6"/>
-    <xacro:big_shelf name="zone_a_r4_9" x="26.0" y="-31.6"/>
-    <xacro:big_shelf name="zone_a_r4_10" x="34.0" y="-31.6"/>
-    <xacro:big_shelf name="zone_a_r4_11" x="42.0" y="-31.6"/>
-    <xacro:big_shelf name="zone_a_r4_12" x="50.0" y="-31.6"/>
-    <xacro:big_shelf name="zone_a_r5_1" x="-54" y="-28.4"/>
-    <xacro:big_shelf name="zone_a_r5_2" x="-46.0" y="-28.4"/>
-    <xacro:big_shelf name="zone_a_r5_3" x="-38.0" y="-28.4"/>
-    <xacro:big_shelf name="zone_a_r5_4" x="-30.0" y="-28.4"/>
-    <xacro:big_shelf name="zone_a_r5_5" x="-22.0" y="-28.4"/>
-    <xacro:big_shelf name="zone_a_r5_6" x="-14.0" y="-28.4"/>
-    <xacro:big_shelf name="zone_a_r5_7" x="10.0" y="-28.4"/>
-    <xacro:big_shelf name="zone_a_r5_8" x="18.0" y="-28.4"/>
-    <xacro:big_shelf name="zone_a_r5_9" x="26.0" y="-28.4"/>
-    <xacro:big_shelf name="zone_a_r5_10" x="34.0" y="-28.4"/>
-    <xacro:big_shelf name="zone_a_r5_11" x="42.0" y="-28.4"/>
-    <xacro:big_shelf name="zone_a_r5_12" x="50.0" y="-28.4"/>
-    <xacro:big_shelf name="zone_a_r6_1" x="-54" y="-27.2"/>
-    <xacro:big_shelf name="zone_a_r6_2" x="-46.0" y="-27.2"/>
-    <xacro:big_shelf name="zone_a_r6_3" x="-38.0" y="-27.2"/>
-    <xacro:big_shelf name="zone_a_r6_4" x="-30.0" y="-27.2"/>
-    <xacro:big_shelf name="zone_a_r6_5" x="-22.0" y="-27.2"/>
-    <xacro:big_shelf name="zone_a_r6_6" x="-14.0" y="-27.2"/>
-    <xacro:big_shelf name="zone_a_r6_7" x="10.0" y="-27.2"/>
-    <xacro:big_shelf name="zone_a_r6_8" x="18.0" y="-27.2"/>
-    <xacro:big_shelf name="zone_a_r6_9" x="26.0" y="-27.2"/>
-    <xacro:big_shelf name="zone_a_r6_10" x="34.0" y="-27.2"/>
-    <xacro:big_shelf name="zone_a_r6_11" x="42.0" y="-27.2"/>
-    <xacro:big_shelf name="zone_a_r6_12" x="50.0" y="-27.2"/>
-    <xacro:big_shelf name="zone_a_r7_1" x="-54" y="-22.0"/>
-    <xacro:big_shelf name="zone_a_r7_2" x="-46.0" y="-22.0"/>
-    <xacro:big_shelf name="zone_a_r7_3" x="-38.0" y="-22.0"/>
-    <xacro:big_shelf name="zone_a_r7_4" x="-30.0" y="-22.0"/>
-    <xacro:big_shelf name="zone_a_r7_5" x="-22.0" y="-22.0"/>
-    <xacro:big_shelf name="zone_a_r7_6" x="-14.0" y="-22.0"/>
-    <xacro:big_shelf name="zone_a_r7_7" x="10.0" y="-22.0"/>
-    <xacro:big_shelf name="zone_a_r7_8" x="18.0" y="-22.0"/>
-    <xacro:big_shelf name="zone_a_r7_9" x="26.0" y="-22.0"/>
-    <xacro:big_shelf name="zone_a_r7_10" x="34.0" y="-22.0"/>
-    <xacro:big_shelf name="zone_a_r7_11" x="42.0" y="-22.0"/>
-    <xacro:big_shelf name="zone_a_r7_12" x="50.0" y="-22.0"/>
-    <xacro:big_shelf name="zone_a_r8_1" x="-54" y="-20.8"/>
-    <xacro:big_shelf name="zone_a_r8_2" x="-46.0" y="-20.8"/>
-    <xacro:big_shelf name="zone_a_r8_3" x="-38.0" y="-20.8"/>
-    <xacro:big_shelf name="zone_a_r8_4" x="-30.0" y="-20.8"/>
-    <xacro:big_shelf name="zone_a_r8_5" x="-22.0" y="-20.8"/>
-    <xacro:big_shelf name="zone_a_r8_6" x="-14.0" y="-20.8"/>
-    <xacro:big_shelf name="zone_a_r8_7" x="10.0" y="-20.8"/>
-    <xacro:big_shelf name="zone_a_r8_8" x="18.0" y="-20.8"/>
-    <xacro:big_shelf name="zone_a_r8_9" x="26.0" y="-20.8"/>
-    <xacro:big_shelf name="zone_a_r8_10" x="34.0" y="-20.8"/>
-    <xacro:big_shelf name="zone_a_r8_11" x="42.0" y="-20.8"/>
-    <xacro:big_shelf name="zone_a_r8_12" x="50.0" y="-20.8"/>
-    <xacro:big_shelf name="zone_a_r9_1" x="-54" y="-17.6"/>
-    <xacro:big_shelf name="zone_a_r9_2" x="-46.0" y="-17.6"/>
-    <xacro:big_shelf name="zone_a_r9_3" x="-38.0" y="-17.6"/>
-    <xacro:big_shelf name="zone_a_r9_4" x="-30.0" y="-17.6"/>
-    <xacro:big_shelf name="zone_a_r9_5" x="-22.0" y="-17.6"/>
-    <xacro:big_shelf name="zone_a_r9_6" x="-14.0" y="-17.6"/>
-    <xacro:big_shelf name="zone_a_r9_7" x="10.0" y="-17.6"/>
-    <xacro:big_shelf name="zone_a_r9_8" x="18.0" y="-17.6"/>
-    <xacro:big_shelf name="zone_a_r9_9" x="26.0" y="-17.6"/>
-    <xacro:big_shelf name="zone_a_r9_10" x="34.0" y="-17.6"/>
-    <xacro:big_shelf name="zone_a_r9_11" x="42.0" y="-17.6"/>
-    <xacro:big_shelf name="zone_a_r9_12" x="50.0" y="-17.6"/>
-    <xacro:big_shelf name="zone_a_r10_1" x="-54" y="-16.4"/>
-    <xacro:big_shelf name="zone_a_r10_2" x="-46.0" y="-16.4"/>
-    <xacro:big_shelf name="zone_a_r10_3" x="-38.0" y="-16.4"/>
-    <xacro:big_shelf name="zone_a_r10_4" x="-30.0" y="-16.4"/>
-    <xacro:big_shelf name="zone_a_r10_5" x="-22.0" y="-16.4"/>
-    <xacro:big_shelf name="zone_a_r10_6" x="-14.0" y="-16.4"/>
-    <xacro:big_shelf name="zone_a_r10_7" x="10.0" y="-16.4"/>
-    <xacro:big_shelf name="zone_a_r10_8" x="18.0" y="-16.4"/>
-    <xacro:big_shelf name="zone_a_r10_9" x="26.0" y="-16.4"/>
-    <xacro:big_shelf name="zone_a_r10_10" x="34.0" y="-16.4"/>
-    <xacro:big_shelf name="zone_a_r10_11" x="42.0" y="-16.4"/>
-    <xacro:big_shelf name="zone_a_r10_12" x="50.0" y="-16.4"/>
-    <xacro:big_shelf name="zone_a_r11_1" x="-54" y="-13.2"/>
-    <xacro:big_shelf name="zone_a_r11_2" x="-46.0" y="-13.2"/>
-    <xacro:big_shelf name="zone_a_r11_3" x="-38.0" y="-13.2"/>
-    <xacro:big_shelf name="zone_a_r11_4" x="-30.0" y="-13.2"/>
-    <xacro:big_shelf name="zone_a_r11_5" x="-22.0" y="-13.2"/>
-    <xacro:big_shelf name="zone_a_r11_6" x="-14.0" y="-13.2"/>
-    <xacro:big_shelf name="zone_a_r11_7" x="10.0" y="-13.2"/>
-    <xacro:big_shelf name="zone_a_r11_8" x="18.0" y="-13.2"/>
-    <xacro:big_shelf name="zone_a_r11_9" x="26.0" y="-13.2"/>
-    <xacro:big_shelf name="zone_a_r11_10" x="34.0" y="-13.2"/>
-    <xacro:big_shelf name="zone_a_r11_11" x="42.0" y="-13.2"/>
-    <xacro:big_shelf name="zone_a_r11_12" x="50.0" y="-13.2"/>
-    <xacro:big_shelf name="zone_a_r12_1" x="-54" y="-12.0"/>
-    <xacro:big_shelf name="zone_a_r12_2" x="-46.0" y="-12.0"/>
-    <xacro:big_shelf name="zone_a_r12_3" x="-38.0" y="-12.0"/>
-    <xacro:big_shelf name="zone_a_r12_4" x="-30.0" y="-12.0"/>
-    <xacro:big_shelf name="zone_a_r12_5" x="-22.0" y="-12.0"/>
-    <xacro:big_shelf name="zone_a_r12_6" x="-14.0" y="-12.0"/>
-    <xacro:big_shelf name="zone_a_r12_7" x="10.0" y="-12.0"/>
-    <xacro:big_shelf name="zone_a_r12_8" x="18.0" y="-12.0"/>
-    <xacro:big_shelf name="zone_a_r12_9" x="26.0" y="-12.0"/>
-    <xacro:big_shelf name="zone_a_r12_10" x="34.0" y="-12.0"/>
-    <xacro:big_shelf name="zone_a_r12_11" x="42.0" y="-12.0"/>
-    <xacro:big_shelf name="zone_a_r12_12" x="50.0" y="-12.0"/>
-    <xacro:big_shelf name="zone_a_r13_1" x="-54" y="-8.8"/>
-    <xacro:big_shelf name="zone_a_r13_2" x="-46.0" y="-8.8"/>
-    <xacro:big_shelf name="zone_a_r13_3" x="-38.0" y="-8.8"/>
-    <xacro:big_shelf name="zone_a_r13_4" x="-30.0" y="-8.8"/>
-    <xacro:big_shelf name="zone_a_r13_5" x="-22.0" y="-8.8"/>
-    <xacro:big_shelf name="zone_a_r13_6" x="-14.0" y="-8.8"/>
-    <xacro:big_shelf name="zone_a_r13_7" x="10.0" y="-8.8"/>
-    <xacro:big_shelf name="zone_a_r13_8" x="18.0" y="-8.8"/>
-    <xacro:big_shelf name="zone_a_r13_9" x="26.0" y="-8.8"/>
-    <xacro:big_shelf name="zone_a_r13_10" x="34.0" y="-8.8"/>
-    <xacro:big_shelf name="zone_a_r13_11" x="42.0" y="-8.8"/>
-    <xacro:big_shelf name="zone_a_r13_12" x="50.0" y="-8.8"/>
-    <xacro:big_shelf name="zone_a_r14_1" x="-54" y="-7.6"/>
-    <xacro:big_shelf name="zone_a_r14_2" x="-46.0" y="-7.6"/>
-    <xacro:big_shelf name="zone_a_r14_3" x="-38.0" y="-7.6"/>
-    <xacro:big_shelf name="zone_a_r14_4" x="-30.0" y="-7.6"/>
-    <xacro:big_shelf name="zone_a_r14_5" x="-22.0" y="-7.6"/>
-    <xacro:big_shelf name="zone_a_r14_6" x="-14.0" y="-7.6"/>
-    <xacro:big_shelf name="zone_a_r14_7" x="10.0" y="-7.6"/>
-    <xacro:big_shelf name="zone_a_r14_8" x="18.0" y="-7.6"/>
-    <xacro:big_shelf name="zone_a_r14_9" x="26.0" y="-7.6"/>
-    <xacro:big_shelf name="zone_a_r14_10" x="34.0" y="-7.6"/>
-    <xacro:big_shelf name="zone_a_r14_11" x="42.0" y="-7.6"/>
-    <xacro:big_shelf name="zone_a_r14_12" x="50.0" y="-7.6"/>
-    <!-- zone_a shelves (big): 168 -->
+    <!-- 14 rows x 14 per row, aisle ~2.0m -->
+    <!-- ============================================================ -->
+    <xacro:big_shelf name="zone_a_r1_1" x="-56" y="-37.2"/>
+    <xacro:big_shelf name="zone_a_r1_2" x="-48.0" y="-37.2"/>
+    <xacro:big_shelf name="zone_a_r1_3" x="-40.0" y="-37.2"/>
+    <xacro:big_shelf name="zone_a_r1_4" x="-32.0" y="-37.2"/>
+    <xacro:big_shelf name="zone_a_r1_5" x="-24.0" y="-37.2"/>
+    <xacro:big_shelf name="zone_a_r1_6" x="-16.0" y="-37.2"/>
+    <xacro:big_shelf name="zone_a_r1_7" x="-8.0" y="-37.2"/>
+    <xacro:big_shelf name="zone_a_r1_8" x="8.0" y="-37.2"/>
+    <xacro:big_shelf name="zone_a_r1_9" x="16.0" y="-37.2"/>
+    <xacro:big_shelf name="zone_a_r1_10" x="24.0" y="-37.2"/>
+    <xacro:big_shelf name="zone_a_r1_11" x="32.0" y="-37.2"/>
+    <xacro:big_shelf name="zone_a_r1_12" x="40.0" y="-37.2"/>
+    <xacro:big_shelf name="zone_a_r1_13" x="48.0" y="-37.2"/>
+    <xacro:big_shelf name="zone_a_r1_14" x="56.0" y="-37.2"/>
+    <xacro:big_shelf name="zone_a_r2_1" x="-56" y="-36.0"/>
+    <xacro:big_shelf name="zone_a_r2_2" x="-48.0" y="-36.0"/>
+    <xacro:big_shelf name="zone_a_r2_3" x="-40.0" y="-36.0"/>
+    <xacro:big_shelf name="zone_a_r2_4" x="-32.0" y="-36.0"/>
+    <xacro:big_shelf name="zone_a_r2_5" x="-24.0" y="-36.0"/>
+    <xacro:big_shelf name="zone_a_r2_6" x="-16.0" y="-36.0"/>
+    <xacro:big_shelf name="zone_a_r2_7" x="-8.0" y="-36.0"/>
+    <xacro:big_shelf name="zone_a_r2_8" x="8.0" y="-36.0"/>
+    <xacro:big_shelf name="zone_a_r2_9" x="16.0" y="-36.0"/>
+    <xacro:big_shelf name="zone_a_r2_10" x="24.0" y="-36.0"/>
+    <xacro:big_shelf name="zone_a_r2_11" x="32.0" y="-36.0"/>
+    <xacro:big_shelf name="zone_a_r2_12" x="40.0" y="-36.0"/>
+    <xacro:big_shelf name="zone_a_r2_13" x="48.0" y="-36.0"/>
+    <xacro:big_shelf name="zone_a_r2_14" x="56.0" y="-36.0"/>
+    <xacro:big_shelf name="zone_a_r3_1" x="-56" y="-32.8"/>
+    <xacro:big_shelf name="zone_a_r3_2" x="-48.0" y="-32.8"/>
+    <xacro:big_shelf name="zone_a_r3_3" x="-40.0" y="-32.8"/>
+    <xacro:big_shelf name="zone_a_r3_4" x="-32.0" y="-32.8"/>
+    <xacro:big_shelf name="zone_a_r3_5" x="-24.0" y="-32.8"/>
+    <xacro:big_shelf name="zone_a_r3_6" x="-16.0" y="-32.8"/>
+    <xacro:big_shelf name="zone_a_r3_7" x="-8.0" y="-32.8"/>
+    <xacro:big_shelf name="zone_a_r3_8" x="8.0" y="-32.8"/>
+    <xacro:big_shelf name="zone_a_r3_9" x="16.0" y="-32.8"/>
+    <xacro:big_shelf name="zone_a_r3_10" x="24.0" y="-32.8"/>
+    <xacro:big_shelf name="zone_a_r3_11" x="32.0" y="-32.8"/>
+    <xacro:big_shelf name="zone_a_r3_12" x="40.0" y="-32.8"/>
+    <xacro:big_shelf name="zone_a_r3_13" x="48.0" y="-32.8"/>
+    <xacro:big_shelf name="zone_a_r3_14" x="56.0" y="-32.8"/>
+    <xacro:big_shelf name="zone_a_r4_1" x="-56" y="-31.6"/>
+    <xacro:big_shelf name="zone_a_r4_2" x="-48.0" y="-31.6"/>
+    <xacro:big_shelf name="zone_a_r4_3" x="-40.0" y="-31.6"/>
+    <xacro:big_shelf name="zone_a_r4_4" x="-32.0" y="-31.6"/>
+    <xacro:big_shelf name="zone_a_r4_5" x="-24.0" y="-31.6"/>
+    <xacro:big_shelf name="zone_a_r4_6" x="-16.0" y="-31.6"/>
+    <xacro:big_shelf name="zone_a_r4_7" x="-8.0" y="-31.6"/>
+    <xacro:big_shelf name="zone_a_r4_8" x="8.0" y="-31.6"/>
+    <xacro:big_shelf name="zone_a_r4_9" x="16.0" y="-31.6"/>
+    <xacro:big_shelf name="zone_a_r4_10" x="24.0" y="-31.6"/>
+    <xacro:big_shelf name="zone_a_r4_11" x="32.0" y="-31.6"/>
+    <xacro:big_shelf name="zone_a_r4_12" x="40.0" y="-31.6"/>
+    <xacro:big_shelf name="zone_a_r4_13" x="48.0" y="-31.6"/>
+    <xacro:big_shelf name="zone_a_r4_14" x="56.0" y="-31.6"/>
+    <xacro:big_shelf name="zone_a_r5_1" x="-56" y="-28.4"/>
+    <xacro:big_shelf name="zone_a_r5_2" x="-48.0" y="-28.4"/>
+    <xacro:big_shelf name="zone_a_r5_3" x="-40.0" y="-28.4"/>
+    <xacro:big_shelf name="zone_a_r5_4" x="-32.0" y="-28.4"/>
+    <xacro:big_shelf name="zone_a_r5_5" x="-24.0" y="-28.4"/>
+    <xacro:big_shelf name="zone_a_r5_6" x="-16.0" y="-28.4"/>
+    <xacro:big_shelf name="zone_a_r5_7" x="-8.0" y="-28.4"/>
+    <xacro:big_shelf name="zone_a_r5_8" x="8.0" y="-28.4"/>
+    <xacro:big_shelf name="zone_a_r5_9" x="16.0" y="-28.4"/>
+    <xacro:big_shelf name="zone_a_r5_10" x="24.0" y="-28.4"/>
+    <xacro:big_shelf name="zone_a_r5_11" x="32.0" y="-28.4"/>
+    <xacro:big_shelf name="zone_a_r5_12" x="40.0" y="-28.4"/>
+    <xacro:big_shelf name="zone_a_r5_13" x="48.0" y="-28.4"/>
+    <xacro:big_shelf name="zone_a_r5_14" x="56.0" y="-28.4"/>
+    <xacro:big_shelf name="zone_a_r6_1" x="-56" y="-27.2"/>
+    <xacro:big_shelf name="zone_a_r6_2" x="-48.0" y="-27.2"/>
+    <xacro:big_shelf name="zone_a_r6_3" x="-40.0" y="-27.2"/>
+    <xacro:big_shelf name="zone_a_r6_4" x="-32.0" y="-27.2"/>
+    <xacro:big_shelf name="zone_a_r6_5" x="-24.0" y="-27.2"/>
+    <xacro:big_shelf name="zone_a_r6_6" x="-16.0" y="-27.2"/>
+    <xacro:big_shelf name="zone_a_r6_7" x="-8.0" y="-27.2"/>
+    <xacro:big_shelf name="zone_a_r6_8" x="8.0" y="-27.2"/>
+    <xacro:big_shelf name="zone_a_r6_9" x="16.0" y="-27.2"/>
+    <xacro:big_shelf name="zone_a_r6_10" x="24.0" y="-27.2"/>
+    <xacro:big_shelf name="zone_a_r6_11" x="32.0" y="-27.2"/>
+    <xacro:big_shelf name="zone_a_r6_12" x="40.0" y="-27.2"/>
+    <xacro:big_shelf name="zone_a_r6_13" x="48.0" y="-27.2"/>
+    <xacro:big_shelf name="zone_a_r6_14" x="56.0" y="-27.2"/>
+    <xacro:big_shelf name="zone_a_r7_1" x="-56" y="-22.0"/>
+    <xacro:big_shelf name="zone_a_r7_2" x="-48.0" y="-22.0"/>
+    <xacro:big_shelf name="zone_a_r7_3" x="-40.0" y="-22.0"/>
+    <xacro:big_shelf name="zone_a_r7_4" x="-32.0" y="-22.0"/>
+    <xacro:big_shelf name="zone_a_r7_5" x="-24.0" y="-22.0"/>
+    <xacro:big_shelf name="zone_a_r7_6" x="-16.0" y="-22.0"/>
+    <xacro:big_shelf name="zone_a_r7_7" x="-8.0" y="-22.0"/>
+    <xacro:big_shelf name="zone_a_r7_8" x="8.0" y="-22.0"/>
+    <xacro:big_shelf name="zone_a_r7_9" x="16.0" y="-22.0"/>
+    <xacro:big_shelf name="zone_a_r7_10" x="24.0" y="-22.0"/>
+    <xacro:big_shelf name="zone_a_r7_11" x="32.0" y="-22.0"/>
+    <xacro:big_shelf name="zone_a_r7_12" x="40.0" y="-22.0"/>
+    <xacro:big_shelf name="zone_a_r7_13" x="48.0" y="-22.0"/>
+    <xacro:big_shelf name="zone_a_r7_14" x="56.0" y="-22.0"/>
+    <xacro:big_shelf name="zone_a_r8_1" x="-56" y="-20.8"/>
+    <xacro:big_shelf name="zone_a_r8_2" x="-48.0" y="-20.8"/>
+    <xacro:big_shelf name="zone_a_r8_3" x="-40.0" y="-20.8"/>
+    <xacro:big_shelf name="zone_a_r8_4" x="-32.0" y="-20.8"/>
+    <xacro:big_shelf name="zone_a_r8_5" x="-24.0" y="-20.8"/>
+    <xacro:big_shelf name="zone_a_r8_6" x="-16.0" y="-20.8"/>
+    <xacro:big_shelf name="zone_a_r8_7" x="-8.0" y="-20.8"/>
+    <xacro:big_shelf name="zone_a_r8_8" x="8.0" y="-20.8"/>
+    <xacro:big_shelf name="zone_a_r8_9" x="16.0" y="-20.8"/>
+    <xacro:big_shelf name="zone_a_r8_10" x="24.0" y="-20.8"/>
+    <xacro:big_shelf name="zone_a_r8_11" x="32.0" y="-20.8"/>
+    <xacro:big_shelf name="zone_a_r8_12" x="40.0" y="-20.8"/>
+    <xacro:big_shelf name="zone_a_r8_13" x="48.0" y="-20.8"/>
+    <xacro:big_shelf name="zone_a_r8_14" x="56.0" y="-20.8"/>
+    <xacro:big_shelf name="zone_a_r9_1" x="-56" y="-17.6"/>
+    <xacro:big_shelf name="zone_a_r9_2" x="-48.0" y="-17.6"/>
+    <xacro:big_shelf name="zone_a_r9_3" x="-40.0" y="-17.6"/>
+    <xacro:big_shelf name="zone_a_r9_4" x="-32.0" y="-17.6"/>
+    <xacro:big_shelf name="zone_a_r9_5" x="-24.0" y="-17.6"/>
+    <xacro:big_shelf name="zone_a_r9_6" x="-16.0" y="-17.6"/>
+    <xacro:big_shelf name="zone_a_r9_7" x="-8.0" y="-17.6"/>
+    <xacro:big_shelf name="zone_a_r9_8" x="8.0" y="-17.6"/>
+    <xacro:big_shelf name="zone_a_r9_9" x="16.0" y="-17.6"/>
+    <xacro:big_shelf name="zone_a_r9_10" x="24.0" y="-17.6"/>
+    <xacro:big_shelf name="zone_a_r9_11" x="32.0" y="-17.6"/>
+    <xacro:big_shelf name="zone_a_r9_12" x="40.0" y="-17.6"/>
+    <xacro:big_shelf name="zone_a_r9_13" x="48.0" y="-17.6"/>
+    <xacro:big_shelf name="zone_a_r9_14" x="56.0" y="-17.6"/>
+    <xacro:big_shelf name="zone_a_r10_1" x="-56" y="-16.4"/>
+    <xacro:big_shelf name="zone_a_r10_2" x="-48.0" y="-16.4"/>
+    <xacro:big_shelf name="zone_a_r10_3" x="-40.0" y="-16.4"/>
+    <xacro:big_shelf name="zone_a_r10_4" x="-32.0" y="-16.4"/>
+    <xacro:big_shelf name="zone_a_r10_5" x="-24.0" y="-16.4"/>
+    <xacro:big_shelf name="zone_a_r10_6" x="-16.0" y="-16.4"/>
+    <xacro:big_shelf name="zone_a_r10_7" x="-8.0" y="-16.4"/>
+    <xacro:big_shelf name="zone_a_r10_8" x="8.0" y="-16.4"/>
+    <xacro:big_shelf name="zone_a_r10_9" x="16.0" y="-16.4"/>
+    <xacro:big_shelf name="zone_a_r10_10" x="24.0" y="-16.4"/>
+    <xacro:big_shelf name="zone_a_r10_11" x="32.0" y="-16.4"/>
+    <xacro:big_shelf name="zone_a_r10_12" x="40.0" y="-16.4"/>
+    <xacro:big_shelf name="zone_a_r10_13" x="48.0" y="-16.4"/>
+    <xacro:big_shelf name="zone_a_r10_14" x="56.0" y="-16.4"/>
+    <xacro:big_shelf name="zone_a_r11_1" x="-56" y="-13.2"/>
+    <xacro:big_shelf name="zone_a_r11_2" x="-48.0" y="-13.2"/>
+    <xacro:big_shelf name="zone_a_r11_3" x="-40.0" y="-13.2"/>
+    <xacro:big_shelf name="zone_a_r11_4" x="-32.0" y="-13.2"/>
+    <xacro:big_shelf name="zone_a_r11_5" x="-24.0" y="-13.2"/>
+    <xacro:big_shelf name="zone_a_r11_6" x="-16.0" y="-13.2"/>
+    <xacro:big_shelf name="zone_a_r11_7" x="-8.0" y="-13.2"/>
+    <xacro:big_shelf name="zone_a_r11_8" x="8.0" y="-13.2"/>
+    <xacro:big_shelf name="zone_a_r11_9" x="16.0" y="-13.2"/>
+    <xacro:big_shelf name="zone_a_r11_10" x="24.0" y="-13.2"/>
+    <xacro:big_shelf name="zone_a_r11_11" x="32.0" y="-13.2"/>
+    <xacro:big_shelf name="zone_a_r11_12" x="40.0" y="-13.2"/>
+    <xacro:big_shelf name="zone_a_r11_13" x="48.0" y="-13.2"/>
+    <xacro:big_shelf name="zone_a_r11_14" x="56.0" y="-13.2"/>
+    <xacro:big_shelf name="zone_a_r12_1" x="-56" y="-12.0"/>
+    <xacro:big_shelf name="zone_a_r12_2" x="-48.0" y="-12.0"/>
+    <xacro:big_shelf name="zone_a_r12_3" x="-40.0" y="-12.0"/>
+    <xacro:big_shelf name="zone_a_r12_4" x="-32.0" y="-12.0"/>
+    <xacro:big_shelf name="zone_a_r12_5" x="-24.0" y="-12.0"/>
+    <xacro:big_shelf name="zone_a_r12_6" x="-16.0" y="-12.0"/>
+    <xacro:big_shelf name="zone_a_r12_7" x="-8.0" y="-12.0"/>
+    <xacro:big_shelf name="zone_a_r12_8" x="8.0" y="-12.0"/>
+    <xacro:big_shelf name="zone_a_r12_9" x="16.0" y="-12.0"/>
+    <xacro:big_shelf name="zone_a_r12_10" x="24.0" y="-12.0"/>
+    <xacro:big_shelf name="zone_a_r12_11" x="32.0" y="-12.0"/>
+    <xacro:big_shelf name="zone_a_r12_12" x="40.0" y="-12.0"/>
+    <xacro:big_shelf name="zone_a_r12_13" x="48.0" y="-12.0"/>
+    <xacro:big_shelf name="zone_a_r12_14" x="56.0" y="-12.0"/>
+    <xacro:big_shelf name="zone_a_r13_1" x="-56" y="-8.8"/>
+    <xacro:big_shelf name="zone_a_r13_2" x="-48.0" y="-8.8"/>
+    <xacro:big_shelf name="zone_a_r13_3" x="-40.0" y="-8.8"/>
+    <xacro:big_shelf name="zone_a_r13_4" x="-32.0" y="-8.8"/>
+    <xacro:big_shelf name="zone_a_r13_5" x="-24.0" y="-8.8"/>
+    <xacro:big_shelf name="zone_a_r13_6" x="-16.0" y="-8.8"/>
+    <xacro:big_shelf name="zone_a_r13_7" x="-8.0" y="-8.8"/>
+    <xacro:big_shelf name="zone_a_r13_8" x="8.0" y="-8.8"/>
+    <xacro:big_shelf name="zone_a_r13_9" x="16.0" y="-8.8"/>
+    <xacro:big_shelf name="zone_a_r13_10" x="24.0" y="-8.8"/>
+    <xacro:big_shelf name="zone_a_r13_11" x="32.0" y="-8.8"/>
+    <xacro:big_shelf name="zone_a_r13_12" x="40.0" y="-8.8"/>
+    <xacro:big_shelf name="zone_a_r13_13" x="48.0" y="-8.8"/>
+    <xacro:big_shelf name="zone_a_r13_14" x="56.0" y="-8.8"/>
+    <xacro:big_shelf name="zone_a_r14_1" x="-56" y="-7.6"/>
+    <xacro:big_shelf name="zone_a_r14_2" x="-48.0" y="-7.6"/>
+    <xacro:big_shelf name="zone_a_r14_3" x="-40.0" y="-7.6"/>
+    <xacro:big_shelf name="zone_a_r14_4" x="-32.0" y="-7.6"/>
+    <xacro:big_shelf name="zone_a_r14_5" x="-24.0" y="-7.6"/>
+    <xacro:big_shelf name="zone_a_r14_6" x="-16.0" y="-7.6"/>
+    <xacro:big_shelf name="zone_a_r14_7" x="-8.0" y="-7.6"/>
+    <xacro:big_shelf name="zone_a_r14_8" x="8.0" y="-7.6"/>
+    <xacro:big_shelf name="zone_a_r14_9" x="16.0" y="-7.6"/>
+    <xacro:big_shelf name="zone_a_r14_10" x="24.0" y="-7.6"/>
+    <xacro:big_shelf name="zone_a_r14_11" x="32.0" y="-7.6"/>
+    <xacro:big_shelf name="zone_a_r14_12" x="40.0" y="-7.6"/>
+    <xacro:big_shelf name="zone_a_r14_13" x="48.0" y="-7.6"/>
+    <xacro:big_shelf name="zone_a_r14_14" x="56.0" y="-7.6"/>
+    <!-- zone_a shelves (big): 196 -->
     <!-- ============================================================ -->
     <!-- ZONE B-WEST: STANDARD (big shelves, back-to-back pairs, 1.6 m aisles) -->
-    <!-- 8 rows x 6 per row, aisle ~1.6m -->
-    <!-- ============================================================ -->
-    <xacro:big_shelf name="zone_bw_r1_1" x="-54" y="4.0"/>
-    <xacro:big_shelf name="zone_bw_r1_2" x="-46.0" y="4.0"/>
-    <xacro:big_shelf name="zone_bw_r1_3" x="-38.0" y="4.0"/>
-    <xacro:big_shelf name="zone_bw_r1_4" x="-30.0" y="4.0"/>
-    <xacro:big_shelf name="zone_bw_r1_5" x="-22.0" y="4.0"/>
-    <xacro:big_shelf name="zone_bw_r1_6" x="-14.0" y="4.0"/>
-    <xacro:big_shelf name="zone_bw_r2_1" x="-54" y="5.2"/>
-    <xacro:big_shelf name="zone_bw_r2_2" x="-46.0" y="5.2"/>
-    <xacro:big_shelf name="zone_bw_r2_3" x="-38.0" y="5.2"/>
-    <xacro:big_shelf name="zone_bw_r2_4" x="-30.0" y="5.2"/>
-    <xacro:big_shelf name="zone_bw_r2_5" x="-22.0" y="5.2"/>
-    <xacro:big_shelf name="zone_bw_r2_6" x="-14.0" y="5.2"/>
-    <xacro:big_shelf name="zone_bw_r3_1" x="-54" y="8.0"/>
-    <xacro:big_shelf name="zone_bw_r3_2" x="-46.0" y="8.0"/>
-    <xacro:big_shelf name="zone_bw_r3_3" x="-38.0" y="8.0"/>
-    <xacro:big_shelf name="zone_bw_r3_4" x="-30.0" y="8.0"/>
-    <xacro:big_shelf name="zone_bw_r3_5" x="-22.0" y="8.0"/>
-    <xacro:big_shelf name="zone_bw_r3_6" x="-14.0" y="8.0"/>
-    <xacro:big_shelf name="zone_bw_r4_1" x="-54" y="9.2"/>
-    <xacro:big_shelf name="zone_bw_r4_2" x="-46.0" y="9.2"/>
-    <xacro:big_shelf name="zone_bw_r4_3" x="-38.0" y="9.2"/>
-    <xacro:big_shelf name="zone_bw_r4_4" x="-30.0" y="9.2"/>
-    <xacro:big_shelf name="zone_bw_r4_5" x="-22.0" y="9.2"/>
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