Commit message: sim robot setup
Signed-off-by: SteveMacenski <stevenmacenski@gmail.com>

File: opennav_benchmark_robot/urdf/benchmark_robot.sdf.xacro (robot description, xacro)
@@ -153,8 +153,8 @@
       </joint>
     </xacro:macro>
-    <xacro:caster_sdf name="front_left" x="0.45" y="0.30"/>
-    <xacro:caster_sdf name="front_right" x="0.45" y="-0.30"/>
-    <xacro:caster_sdf name="rear_left" x="-0.45" y="0.30"/>
-    <xacro:caster_sdf name="rear_right" x="-0.45" y="-0.30"/>
+    <xacro:caster_sdf name="rear_left" x="0.45" y="0.30"/>
+    <xacro:caster_sdf name="rear_right" x="0.45" y="-0.30"/>
+    <xacro:caster_sdf name="front_left" x="-0.45" y="0.30"/>
+    <xacro:caster_sdf name="front_right" x="-0.45" y="-0.30"/>
     <!-- ============ IMU ============ -->
     <link name="imu_link">
@@ -191,8 +191,8 @@
       <child>imu_link</child>
     </joint>
-    <!-- ============ 3D LIDARS (mounted on sensor tower) ============ -->
-    <!-- Center: top of tower, 360deg, 32ch, 75m -->
+    <!-- ============ 3D LIDARS ============ -->
+    <!-- Center: 360deg, 32ch -->
     <link name="lidar_3d_center_link">
-      <pose relative_to="sensor_tower_link">0 0 0.167 0 0 0</pose>
+      <pose relative_to="base_link">0.10 0 0.825 0 0 0</pose>
       <inertial>
         <mass>0.5</mass>
@@ -248,10 +248,10 @@
     </link>
     <joint name="lidar_3d_center_joint" type="fixed">
-      <parent>sensor_tower_link</parent>
+      <parent>base_link</parent>
       <child>lidar_3d_center_link</child>
     </joint>
-    <!-- Front-left: on left arm, 120deg, 16ch, 30m, tilted down 15deg -->
-    <link name="lidar_3d_front_left_link">
-      <pose relative_to="sensor_tower_link">0 0.24 0.148 -0.2618 0 0</pose>
+    <!-- Top: on tower surface, in front of center lidar -->
+    <link name="lidar_3d_top_link">
+      <pose relative_to="base_link">0.35 0 2.195 0 0 0</pose>
       <inertial>
         <mass>0.5</mass>
@@ -272,5 +272,5 @@
         </material>
       </visual>
-      <sensor name="lidar_3d_front_left_sensor" type="gpu_lidar">
+      <sensor name="lidar_3d_top_sensor" type="gpu_lidar">
         <always_on>true</always_on>
         <update_rate>10</update_rate>
@@ -301,16 +301,16 @@
           </noise>
         </lidar>
-        <topic>${ns}/lidar_3d_front_left/points</topic>
-        <gz_frame_id>lidar_3d_front_left_link</gz_frame_id>
+        <topic>${ns}/lidar_3d_top/points</topic>
+        <gz_frame_id>lidar_3d_top_link</gz_frame_id>
         <visibility_mask>${lidar_visibility_mask}</visibility_mask>
       </sensor>
     </link>
-    <joint name="lidar_3d_front_left_joint" type="fixed">
-      <parent>sensor_tower_link</parent>
-      <child>lidar_3d_front_left_link</child>
-    </joint>
-    <!-- Front-right: on right arm, 120deg, 16ch, 30m, tilted down 15deg -->
-    <link name="lidar_3d_front_right_link">
-      <pose relative_to="sensor_tower_link">0 -0.24 0.148 0.2618 0 0</pose>
+    <joint name="lidar_3d_top_joint" type="fixed">
+      <parent>base_link</parent>
+      <child>lidar_3d_top_link</child>
+    </joint>
+    <!-- Front-right: 16ch, tilted down 15deg -->
+    <link name="lidar_3d_tilted_link">
+      <pose relative_to="base_link">0.10 0 1.845 0.7854 0 1.5708</pose>
       <inertial>
         <mass>0.5</mass>
@@ -331,5 +331,5 @@
         </material>
       </visual>
-      <sensor name="lidar_3d_front_right_sensor" type="gpu_lidar">
+      <sensor name="lidar_3d_tilted_sensor" type="gpu_lidar">
         <always_on>true</always_on>
         <update_rate>10</update_rate>
@@ -360,16 +360,16 @@
           </noise>
         </lidar>
-        <topic>${ns}/lidar_3d_front_right/points</topic>
-        <gz_frame_id>lidar_3d_front_right_link</gz_frame_id>
+        <topic>${ns}/lidar_3d_tilted/points</topic>
+        <gz_frame_id>lidar_3d_tilted_link</gz_frame_id>
         <visibility_mask>${lidar_visibility_mask}</visibility_mask>
       </sensor>
     </link>
-    <joint name="lidar_3d_front_right_joint" type="fixed">
-      <parent>sensor_tower_link</parent>
-      <child>lidar_3d_front_right_link</child>
+    <joint name="lidar_3d_tilted_joint" type="fixed">
+      <parent>base_link</parent>
+      <child>lidar_3d_tilted_link</child>
     </joint>
     <!-- ============ 2D LIDARS (SICK TiM781 on chassis corners) ============ -->
-    <link name="lidar_2d_front_link">
-      <pose relative_to="base_link">0.50 0.30 0.13 0 0 0.7854</pose>
+    <link name="lidar_2d_front_left_link">
+      <pose relative_to="base_link">-0.50 0.40 0.60 0 0 2.356</pose>
       <inertial>
         <mass>0.4</mass>
@@ -390,5 +390,5 @@
         </material>
       </visual>
-      <sensor name="lidar_2d_front_sensor" type="gpu_lidar">
+      <sensor name="lidar_2d_front_left_sensor" type="gpu_lidar">
         <always_on>true</always_on>
         <update_rate>30</update_rate>
@@ -419,15 +419,15 @@
           </noise>
         </lidar>
-        <topic>${ns}/scan_front</topic>
-        <gz_frame_id>lidar_2d_front_link</gz_frame_id>
+        <topic>${ns}/scan_front_left</topic>
+        <gz_frame_id>lidar_2d_front_left_link</gz_frame_id>
         <visibility_mask>${lidar_visibility_mask}</visibility_mask>
       </sensor>
     </link>
-    <joint name="lidar_2d_front_joint" type="fixed">
-      <parent>base_link</parent>
-      <child>lidar_2d_front_link</child>
-    </joint>
-    <link name="lidar_2d_rear_link">
-      <pose relative_to="base_link">-0.50 -0.30 0.13 0 0 -2.356</pose>
+    <joint name="lidar_2d_front_left_joint" type="fixed">
+      <parent>base_link</parent>
+      <child>lidar_2d_front_left_link</child>
+    </joint>
+    <link name="lidar_2d_front_right_link">
+      <pose relative_to="base_link">-0.50 -0.40 0.60 0 0 -2.356</pose>
       <inertial>
         <mass>0.4</mass>
@@ -448,5 +448,5 @@
         </material>
       </visual>
-      <sensor name="lidar_2d_rear_sensor" type="gpu_lidar">
+      <sensor name="lidar_2d_front_right_sensor" type="gpu_lidar">
         <always_on>true</always_on>
         <update_rate>30</update_rate>
@@ -477,12 +477,12 @@
           </noise>
         </lidar>
-        <topic>${ns}/scan_rear</topic>
-        <gz_frame_id>lidar_2d_rear_link</gz_frame_id>
+        <topic>${ns}/scan_front_right</topic>
+        <gz_frame_id>lidar_2d_front_right_link</gz_frame_id>
         <visibility_mask>${lidar_visibility_mask}</visibility_mask>
       </sensor>
     </link>
-    <joint name="lidar_2d_rear_joint" type="fixed">
-      <parent>base_link</parent>
-      <child>lidar_2d_rear_link</child>
+    <joint name="lidar_2d_front_right_joint" type="fixed">
+      <parent>base_link</parent>
+      <child>lidar_2d_front_right_link</child>
     </joint>
     <!-- ============ DEPTH CAMERAS (Orbbec Gemini 335 on chassis faces) ============ -->
@@ -531,7 +531,7 @@
       </joint>
     </xacro:macro>
-    <xacro:camera_sdf name="camera_front_left" x="0.60" y="0.20" z="0.05" pitch="0.2618" yaw="-0.5245"/>
-    <xacro:camera_sdf name="camera_front_right" x="0.60" y="-0.20" z="0.05" pitch="0.2618" yaw="0.5245"/>
-    <xacro:camera_sdf name="camera_rear" x="-0.60" y="0" z="0.05" pitch="0" yaw="3.14159"/>
+    <xacro:camera_sdf name="camera_rear" x="0.235" y="0" z="0.175" pitch="0" yaw="0"/>
+    <xacro:camera_sdf name="camera_front_left" x="-0.63" y="0.20" z="0.10" pitch="0.2618" yaw="${3.14159 + 0.5245}"/>
+    <xacro:camera_sdf name="camera_front_right" x="-0.63" y="-0.20" z="0.10" pitch="0.2618" yaw="${3.14159 - 0.5245}"/>
     <!-- ============ PLUGINS ============ -->
     <plugin filename="gz-sim-diff-drive-system" name="gz::sim::systems::DiffDrive">

File: opennav_benchmark_robot/urdf/benchmark_robot.urdf.xacro (robot description, xacro)
@@ -13,7 +13,4 @@
   <xacro:property name="caster_radius" value="0.05"/>
   <xacro:property name="caster_mass" value="0.5"/>
-  <!-- Tower: arc panel at front, bottom aligns with chassis top -->
-  <xacro:property name="tower_x" value="0.52"/>
-  <xacro:property name="tower_z_offset" value="0.318"/>
   <!-- Colors -->
   <material name="nav2_blue">
@@ -77,17 +74,4 @@
     <child link="base_link"/>
     <origin xyz="0 0 ${chassis_z_offset}" rpy="0 0 0"/>
-  </joint>
-  <!-- ============ SENSOR TOWER ============ -->
-  <link name="sensor_tower_link">
-    <!-- sensor_tower visual removed (forklift mesh replaces it) -->
-    <inertial>
-      <mass value="3.0"/>
-      <inertia ixx="0.03" ixy="0" ixz="0" iyy="0.03" iyz="0" izz="0.01"/>
-    </inertial>
-  </link>
-  <joint name="sensor_tower_joint" type="fixed">
-    <parent link="base_link"/>
-    <child link="sensor_tower_link"/>
-    <origin xyz="${tower_x} 0 ${tower_z_offset}" rpy="0 0 0"/>
   </joint>
   <!-- ============ DRIVE WHEELS ============ -->
@@ -140,8 +124,8 @@
     </joint>
   </xacro:macro>
-  <xacro:caster_wheel name="front_left" x="0.45" y="0.30"/>
-  <xacro:caster_wheel name="front_right" x="0.45" y="-0.30"/>
-  <xacro:caster_wheel name="rear_left" x="-0.45" y="0.30"/>
-  <xacro:caster_wheel name="rear_right" x="-0.45" y="-0.30"/>
+  <xacro:caster_wheel name="rear_left" x="0.45" y="0.30"/>
+  <xacro:caster_wheel name="rear_right" x="0.45" y="-0.30"/>
+  <xacro:caster_wheel name="front_left" x="-0.45" y="0.30"/>
+  <xacro:caster_wheel name="front_right" x="-0.45" y="-0.30"/>
   <!-- ============ IMU ============ -->
   <link name="imu_link">
@@ -156,6 +140,6 @@
     <origin xyz="0 0 -0.05" rpy="0 0 0"/>
   </joint>
-  <!-- ============ 3D LIDARS (Ouster OS1-32 on tower) ============ -->
-  <!-- Center: top of tower -->
+  <!-- ============ 3D LIDARS ============ -->
+  <!-- Center: 360deg, 32ch -->
   <link name="lidar_3d_center_link">
     <visual>
@@ -174,10 +158,10 @@
   </link>
   <joint name="lidar_3d_center_joint" type="fixed">
-    <parent link="sensor_tower_link"/>
+    <parent link="base_link"/>
     <child link="lidar_3d_center_link"/>
-    <origin xyz="0 0 0.167" rpy="0 0 0"/>
-  </joint>
-  <!-- Front-left: on left arm of tower crossbar -->
-  <link name="lidar_3d_front_left_link">
+    <origin xyz="0.10 0 0.825" rpy="0 0 0"/>
+  </joint>
+  <!-- Top: on tower surface, in front of center lidar -->
+  <link name="lidar_3d_top_link">
     <visual>
       <geometry>
@@ -194,11 +178,11 @@
     </inertial>
   </link>
-  <joint name="lidar_3d_front_left_joint" type="fixed">
-    <parent link="sensor_tower_link"/>
-    <child link="lidar_3d_front_left_link"/>
-    <origin xyz="0 0.24 0.148" rpy="${-pi/12} 0 0"/>
-  </joint>
-  <!-- Front-right: on right arm of tower crossbar -->
-  <link name="lidar_3d_front_right_link">
+  <joint name="lidar_3d_top_joint" type="fixed">
+    <parent link="base_link"/>
+    <child link="lidar_3d_top_link"/>
+    <origin xyz="0.35 0 2.195" rpy="0 0 0"/>
+  </joint>
+  <!-- Tilted: 16ch, pitched 270deg -->
+  <link name="lidar_3d_tilted_link">
     <visual>
       <geometry>
@@ -215,8 +199,8 @@
     </inertial>
   </link>
-  <joint name="lidar_3d_front_right_joint" type="fixed">
-    <parent link="sensor_tower_link"/>
-    <child link="lidar_3d_front_right_link"/>
-    <origin xyz="0 -0.24 0.148" rpy="${pi/12} 0 0"/>
+  <joint name="lidar_3d_tilted_joint" type="fixed">
+    <parent link="base_link"/>
+    <child link="lidar_3d_tilted_link"/>
+    <origin xyz="0.10 0 1.845" rpy="${pi/4} 0 ${pi/2}"/>
   </joint>
   <!-- ============ 2D LIDARS (SICK TiM781 on chassis corners) ============ -->
@@ -240,9 +224,9 @@
       <parent link="base_link"/>
       <child link="${name}_link"/>
-      <origin xyz="${x} ${y} ${chassis_height/2 - 0.02}" rpy="0 0 ${yaw}"/>
-    </joint>
-  </xacro:macro>
-  <xacro:lidar_2d name="lidar_2d_front" x="0.50" y="0.30" yaw="${pi/4}"/>
-  <xacro:lidar_2d name="lidar_2d_rear" x="-0.50" y="-0.30" yaw="${-3*pi/4}"/>
+      <origin xyz="${x} ${y} ${chassis_height/2 + 0.45}" rpy="0 0 ${yaw}"/>
+    </joint>
+  </xacro:macro>
+  <xacro:lidar_2d name="lidar_2d_front_left" x="-0.50" y="0.40" yaw="${3*pi/4}"/>
+  <xacro:lidar_2d name="lidar_2d_front_right" x="-0.50" y="-0.40" yaw="${-3*pi/4}"/>
   <!-- ============ DEPTH CAMERAS (Orbbec Gemini 335) ============ -->
   <xacro:macro name="depth_camera" params="name x y z pitch yaw">
@@ -274,6 +258,6 @@
     </joint>
   </xacro:macro>
-  <xacro:depth_camera name="camera_front_left" x="0.60" y="0.20" z="0.05" pitch="${pi/12}" yaw="-0.5245"/>
-  <xacro:depth_camera name="camera_front_right" x="0.60" y="-0.20" z="0.05" pitch="${pi/12}" yaw="0.5245"/>
-  <xacro:depth_camera name="camera_rear" x="-0.60" y="0" z="0.05" pitch="0" yaw="${pi}"/>
+  <xacro:depth_camera name="camera_rear" x="0.235" y="0" z="0.175" pitch="0" yaw="0"/>
+  <xacro:depth_camera name="camera_front_left" x="-0.63" y="0.20" z="0.10" pitch="${pi/12}" yaw="${pi + 0.5245}"/>
+  <xacro:depth_camera name="camera_front_right" x="-0.63" y="-0.20" z="0.10" pitch="${pi/12}" yaw="${pi - 0.5245}"/>
 </robot>

Commit message: warehouse incremental inprovements
Signed-off-by: SteveMacenski <stevenmacenski@gmail.com>

File: opennav_benchmark_robot/urdf/benchmark_robot.sdf.xacro (robot description, xacro)
@@ -233,5 +233,5 @@
           <range>
             <min>0.3</min>
-            <max>50.0</max>
+            <max>30.0</max>
             <resolution>0.01</resolution>
           </range>
