Commit message: warehouse incremental inprovements
Signed-off-by: SteveMacenski <stevenmacenski@gmail.com>

File: opennav_benchmark_sim/worlds/benchmark_warehouse.sdf.xacro (robot description, xacro)
@@ -40,13 +40,13 @@
       <direction>-0.3 0.2 -1.0</direction>
     </light>
-    <!-- Ground plane (120m x 140m) -->
+    <!-- Ground plane (128m x 140m) -->
     <model name="ground_plane">
       <static>true</static>
       <link name="link">
         <collision name="collision">
-          <geometry><plane><normal>0 0 1</normal><size>120 140</size></plane></geometry>
+          <geometry><plane><normal>0 0 1</normal><size>128 140</size></plane></geometry>
         </collision>
         <visual name="visual">
-          <geometry><plane><normal>0 0 1</normal><size>120 140</size></plane></geometry>
+          <geometry><plane><normal>0 0 1</normal><size>128 140</size></plane></geometry>
           <material>
             <ambient>0.55 0.55 0.53 1</ambient>
@@ -181,11 +181,11 @@
     </xacro:macro>
     <!-- ============================================================ -->
-    <!-- PERIMETER WALLS (120m x 140m, 10.0m tall brick) -->
-    <!-- ============================================================ -->
-    <xacro:wall_segment name="north" x="0" y="70.0" yaw="0" length="120"/>
-    <xacro:wall_segment name="east" x="60.0" y="0" yaw="1.5708" length="140"/>
-    <xacro:wall_segment name="west" x="-60.0" y="0" yaw="1.5708" length="140"/>
+    <!-- PERIMETER WALLS (128m x 140m, 10.0m tall brick) -->
+    <!-- ============================================================ -->
+    <xacro:wall_segment name="north" x="0" y="70.0" yaw="0" length="128"/>
+    <xacro:wall_segment name="east" x="64.0" y="0" yaw="1.5708" length="140"/>
+    <xacro:wall_segment name="west" x="-64.0" y="0" yaw="1.5708" length="140"/>
     <!-- South wall segments (between dock doors) -->
-    <xacro:wall_segment name="south_1" x="-56.0" y="-70.0" yaw="0" length="8.0"/>
+    <xacro:wall_segment name="south_1" x="-58.0" y="-70.0" yaw="0" length="12.0"/>
     <xacro:wall_segment name="south_2" x="-44.0" y="-70.0" yaw="0" length="8.0"/>
     <xacro:wall_segment name="south_3" x="-32.0" y="-70.0" yaw="0" length="8.0"/>
@@ -195,5 +195,5 @@
     <xacro:wall_segment name="south_7" x="16.0" y="-70.0" yaw="0" length="8.0"/>
     <xacro:wall_segment name="south_8" x="28.0" y="-70.0" yaw="0" length="8.0"/>
-    <xacro:wall_segment name="south_9" x="48.0" y="-70.0" yaw="0" length="24.0"/>
+    <xacro:wall_segment name="south_9" x="50.0" y="-70.0" yaw="0" length="28.0"/>
     <!-- Roll-up dock doors -->
     <xacro:dock_door name="dock1" x="-50" y="-70.0" yaw="0"/>
@@ -222,233 +222,233 @@
     <xacro:support_column name="s12" x="4" y="-70.0"/>
     <xacro:support_column name="s13" x="16" y="-70.0"/>
-    <xacro:support_column name="e14" x="60.0" y="-60"/>
-    <xacro:support_column name="e15" x="60.0" y="-40"/>
-    <xacro:support_column name="e16" x="60.0" y="-20"/>
-    <xacro:support_column name="e17" x="60.0" y="0"/>
-    <xacro:support_column name="e18" x="60.0" y="20"/>
-    <xacro:support_column name="e19" x="60.0" y="40"/>
-    <xacro:support_column name="e20" x="60.0" y="60"/>
-    <xacro:support_column name="w21" x="-60.0" y="-60"/>
-    <xacro:support_column name="w22" x="-60.0" y="-40"/>
-    <xacro:support_column name="w23" x="-60.0" y="-20"/>
-    <xacro:support_column name="w24" x="-60.0" y="0"/>
-    <xacro:support_column name="w25" x="-60.0" y="20"/>
-    <xacro:support_column name="w26" x="-60.0" y="40"/>
-    <xacro:support_column name="w27" x="-60.0" y="60"/>
-    <xacro:support_column name="int_28" x="-40" y="-40"/>
-    <xacro:support_column name="int_29" x="-40" y="-23"/>
-    <xacro:support_column name="int_30" x="-40" y="15"/>
-    <xacro:support_column name="int_31" x="-40" y="40"/>
-    <xacro:support_column name="int_32" x="-20" y="-40"/>
-    <xacro:support_column name="int_33" x="-20" y="-23"/>
-    <xacro:support_column name="int_34" x="-20" y="15"/>
-    <xacro:support_column name="int_35" x="-20" y="40"/>
-    <xacro:support_column name="int_36" x="20" y="-40"/>
-    <xacro:support_column name="int_37" x="20" y="-23"/>
-    <xacro:support_column name="int_38" x="20" y="15"/>
-    <xacro:support_column name="int_39" x="20" y="40"/>
-    <xacro:support_column name="int_40" x="40" y="-40"/>
-    <xacro:support_column name="int_41" x="40" y="-23"/>
-    <xacro:support_column name="int_42" x="40" y="15"/>
+    <xacro:support_column name="e14" x="64.0" y="-60"/>
+    <xacro:support_column name="e15" x="64.0" y="-40"/>
+    <xacro:support_column name="e16" x="64.0" y="-20"/>
+    <xacro:support_column name="e17" x="64.0" y="0"/>
+    <xacro:support_column name="e18" x="64.0" y="20"/>
+    <xacro:support_column name="e19" x="64.0" y="40"/>
+    <xacro:support_column name="e20" x="64.0" y="60"/>
+    <xacro:support_column name="w21" x="-64.0" y="-60"/>
+    <xacro:support_column name="w22" x="-64.0" y="-40"/>
+    <xacro:support_column name="w23" x="-64.0" y="-20"/>
+    <xacro:support_column name="w24" x="-64.0" y="0"/>
+    <xacro:support_column name="w25" x="-64.0" y="20"/>
+    <xacro:support_column name="w26" x="-64.0" y="40"/>
+    <xacro:support_column name="w27" x="-64.0" y="60"/>
+    <xacro:support_column name="int_28" x="-38.0" y="-40"/>
+    <xacro:support_column name="int_29" x="-38.0" y="-23"/>
+    <xacro:support_column name="int_30" x="-38.0" y="15"/>
+    <xacro:support_column name="int_31" x="-38.0" y="40"/>
+    <xacro:support_column name="int_32" x="-18.0" y="-40"/>
+    <xacro:support_column name="int_33" x="-18.0" y="-23"/>
+    <xacro:support_column name="int_34" x="-18.0" y="15"/>
+    <xacro:support_column name="int_35" x="-18.0" y="40"/>
+    <xacro:support_column name="int_36" x="22.0" y="-40"/>
+    <xacro:support_column name="int_37" x="22.0" y="-23"/>
+    <xacro:support_column name="int_38" x="22.0" y="15"/>
+    <xacro:support_column name="int_39" x="22.0" y="40"/>
+    <xacro:support_column name="int_40" x="42.0" y="-40"/>
+    <xacro:support_column name="int_41" x="42.0" y="-23"/>
+    <xacro:support_column name="int_42" x="42.0" y="15"/>
     <!-- ============================================================ -->
     <!-- ZONE A: BULK STORAGE (big shelves, back-to-back pairs, 2.0 m aisles) -->
     <!-- 14 rows x 14 per row, aisle ~2.0m -->
     <!-- ============================================================ -->
-    <xacro:big_shelf name="zone_a_r1_1" x="-56" y="-37.2"/>
-    <xacro:big_shelf name="zone_a_r1_2" x="-48.0" y="-37.2"/>
-    <xacro:big_shelf name="zone_a_r1_3" x="-40.0" y="-37.2"/>
-    <xacro:big_shelf name="zone_a_r1_4" x="-32.0" y="-37.2"/>
-    <xacro:big_shelf name="zone_a_r1_5" x="-24.0" y="-37.2"/>
-    <xacro:big_shelf name="zone_a_r1_6" x="-16.0" y="-37.2"/>
-    <xacro:big_shelf name="zone_a_r1_7" x="-8.0" y="-37.2"/>
-    <xacro:big_shelf name="zone_a_r1_8" x="8.0" y="-37.2"/>
-    <xacro:big_shelf name="zone_a_r1_9" x="16.0" y="-37.2"/>
-    <xacro:big_shelf name="zone_a_r1_10" x="24.0" y="-37.2"/>
-    <xacro:big_shelf name="zone_a_r1_11" x="32.0" y="-37.2"/>
-    <xacro:big_shelf name="zone_a_r1_12" x="40.0" y="-37.2"/>
-    <xacro:big_shelf name="zone_a_r1_13" x="48.0" y="-37.2"/>
-    <xacro:big_shelf name="zone_a_r1_14" x="56.0" y="-37.2"/>
-    <xacro:big_shelf name="zone_a_r2_1" x="-56" y="-36.0"/>
-    <xacro:big_shelf name="zone_a_r2_2" x="-48.0" y="-36.0"/>
-    <xacro:big_shelf name="zone_a_r2_3" x="-40.0" y="-36.0"/>
-    <xacro:big_shelf name="zone_a_r2_4" x="-32.0" y="-36.0"/>
-    <xacro:big_shelf name="zone_a_r2_5" x="-24.0" y="-36.0"/>
-    <xacro:big_shelf name="zone_a_r2_6" x="-16.0" y="-36.0"/>
-    <xacro:big_shelf name="zone_a_r2_7" x="-8.0" y="-36.0"/>
-    <xacro:big_shelf name="zone_a_r2_8" x="8.0" y="-36.0"/>
-    <xacro:big_shelf name="zone_a_r2_9" x="16.0" y="-36.0"/>
-    <xacro:big_shelf name="zone_a_r2_10" x="24.0" y="-36.0"/>
-    <xacro:big_shelf name="zone_a_r2_11" x="32.0" y="-36.0"/>
-    <xacro:big_shelf name="zone_a_r2_12" x="40.0" y="-36.0"/>
-    <xacro:big_shelf name="zone_a_r2_13" x="48.0" y="-36.0"/>
-    <xacro:big_shelf name="zone_a_r2_14" x="56.0" y="-36.0"/>
-    <xacro:big_shelf name="zone_a_r3_1" x="-56" y="-32.8"/>
-    <xacro:big_shelf name="zone_a_r3_2" x="-48.0" y="-32.8"/>
-    <xacro:big_shelf name="zone_a_r3_3" x="-40.0" y="-32.8"/>
-    <xacro:big_shelf name="zone_a_r3_4" x="-32.0" y="-32.8"/>
-    <xacro:big_shelf name="zone_a_r3_5" x="-24.0" y="-32.8"/>
-    <xacro:big_shelf name="zone_a_r3_6" x="-16.0" y="-32.8"/>
-    <xacro:big_shelf name="zone_a_r3_7" x="-8.0" y="-32.8"/>
-    <xacro:big_shelf name="zone_a_r3_8" x="8.0" y="-32.8"/>
-    <xacro:big_shelf name="zone_a_r3_9" x="16.0" y="-32.8"/>
-    <xacro:big_shelf name="zone_a_r3_10" x="24.0" y="-32.8"/>
-    <xacro:big_shelf name="zone_a_r3_11" x="32.0" y="-32.8"/>
-    <xacro:big_shelf name="zone_a_r3_12" x="40.0" y="-32.8"/>
-    <xacro:big_shelf name="zone_a_r3_13" x="48.0" y="-32.8"/>
-    <xacro:big_shelf name="zone_a_r3_14" x="56.0" y="-32.8"/>
-    <xacro:big_shelf name="zone_a_r4_1" x="-56" y="-31.6"/>
-    <xacro:big_shelf name="zone_a_r4_2" x="-48.0" y="-31.6"/>
-    <xacro:big_shelf name="zone_a_r4_3" x="-40.0" y="-31.6"/>
-    <xacro:big_shelf name="zone_a_r4_4" x="-32.0" y="-31.6"/>
-    <xacro:big_shelf name="zone_a_r4_5" x="-24.0" y="-31.6"/>
-    <xacro:big_shelf name="zone_a_r4_6" x="-16.0" y="-31.6"/>
-    <xacro:big_shelf name="zone_a_r4_7" x="-8.0" y="-31.6"/>
-    <xacro:big_shelf name="zone_a_r4_8" x="8.0" y="-31.6"/>
-    <xacro:big_shelf name="zone_a_r4_9" x="16.0" y="-31.6"/>
-    <xacro:big_shelf name="zone_a_r4_10" x="24.0" y="-31.6"/>
-    <xacro:big_shelf name="zone_a_r4_11" x="32.0" y="-31.6"/>
-    <xacro:big_shelf name="zone_a_r4_12" x="40.0" y="-31.6"/>
-    <xacro:big_shelf name="zone_a_r4_13" x="48.0" y="-31.6"/>
-    <xacro:big_shelf name="zone_a_r4_14" x="56.0" y="-31.6"/>
-    <xacro:big_shelf name="zone_a_r5_1" x="-56" y="-28.4"/>
-    <xacro:big_shelf name="zone_a_r5_2" x="-48.0" y="-28.4"/>
-    <xacro:big_shelf name="zone_a_r5_3" x="-40.0" y="-28.4"/>
-    <xacro:big_shelf name="zone_a_r5_4" x="-32.0" y="-28.4"/>
-    <xacro:big_shelf name="zone_a_r5_5" x="-24.0" y="-28.4"/>
-    <xacro:big_shelf name="zone_a_r5_6" x="-16.0" y="-28.4"/>
-    <xacro:big_shelf name="zone_a_r5_7" x="-8.0" y="-28.4"/>
-    <xacro:big_shelf name="zone_a_r5_8" x="8.0" y="-28.4"/>
-    <xacro:big_shelf name="zone_a_r5_9" x="16.0" y="-28.4"/>
-    <xacro:big_shelf name="zone_a_r5_10" x="24.0" y="-28.4"/>
-    <xacro:big_shelf name="zone_a_r5_11" x="32.0" y="-28.4"/>
-    <xacro:big_shelf name="zone_a_r5_12" x="40.0" y="-28.4"/>
-    <xacro:big_shelf name="zone_a_r5_13" x="48.0" y="-28.4"/>
-    <xacro:big_shelf name="zone_a_r5_14" x="56.0" y="-28.4"/>
-    <xacro:big_shelf name="zone_a_r6_1" x="-56" y="-27.2"/>
-    <xacro:big_shelf name="zone_a_r6_2" x="-48.0" y="-27.2"/>
-    <xacro:big_shelf name="zone_a_r6_3" x="-40.0" y="-27.2"/>
-    <xacro:big_shelf name="zone_a_r6_4" x="-32.0" y="-27.2"/>
-    <xacro:big_shelf name="zone_a_r6_5" x="-24.0" y="-27.2"/>
-    <xacro:big_shelf name="zone_a_r6_6" x="-16.0" y="-27.2"/>
-    <xacro:big_shelf name="zone_a_r6_7" x="-8.0" y="-27.2"/>
-    <xacro:big_shelf name="zone_a_r6_8" x="8.0" y="-27.2"/>
-    <xacro:big_shelf name="zone_a_r6_9" x="16.0" y="-27.2"/>
-    <xacro:big_shelf name="zone_a_r6_10" x="24.0" y="-27.2"/>
-    <xacro:big_shelf name="zone_a_r6_11" x="32.0" y="-27.2"/>
-    <xacro:big_shelf name="zone_a_r6_12" x="40.0" y="-27.2"/>
-    <xacro:big_shelf name="zone_a_r6_13" x="48.0" y="-27.2"/>
-    <xacro:big_shelf name="zone_a_r6_14" x="56.0" y="-27.2"/>
-    <xacro:big_shelf name="zone_a_r7_1" x="-56" y="-22.0"/>
-    <xacro:big_shelf name="zone_a_r7_2" x="-48.0" y="-22.0"/>
-    <xacro:big_shelf name="zone_a_r7_3" x="-40.0" y="-22.0"/>
-    <xacro:big_shelf name="zone_a_r7_4" x="-32.0" y="-22.0"/>
-    <xacro:big_shelf name="zone_a_r7_5" x="-24.0" y="-22.0"/>
-    <xacro:big_shelf name="zone_a_r7_6" x="-16.0" y="-22.0"/>
-    <xacro:big_shelf name="zone_a_r7_7" x="-8.0" y="-22.0"/>
-    <xacro:big_shelf name="zone_a_r7_8" x="8.0" y="-22.0"/>
-    <xacro:big_shelf name="zone_a_r7_9" x="16.0" y="-22.0"/>
-    <xacro:big_shelf name="zone_a_r7_10" x="24.0" y="-22.0"/>
-    <xacro:big_shelf name="zone_a_r7_11" x="32.0" y="-22.0"/>
-    <xacro:big_shelf name="zone_a_r7_12" x="40.0" y="-22.0"/>
-    <xacro:big_shelf name="zone_a_r7_13" x="48.0" y="-22.0"/>
-    <xacro:big_shelf name="zone_a_r7_14" x="56.0" y="-22.0"/>
-    <xacro:big_shelf name="zone_a_r8_1" x="-56" y="-20.8"/>
-    <xacro:big_shelf name="zone_a_r8_2" x="-48.0" y="-20.8"/>
-    <xacro:big_shelf name="zone_a_r8_3" x="-40.0" y="-20.8"/>
-    <xacro:big_shelf name="zone_a_r8_4" x="-32.0" y="-20.8"/>
-    <xacro:big_shelf name="zone_a_r8_5" x="-24.0" y="-20.8"/>
-    <xacro:big_shelf name="zone_a_r8_6" x="-16.0" y="-20.8"/>
-    <xacro:big_shelf name="zone_a_r8_7" x="-8.0" y="-20.8"/>
-    <xacro:big_shelf name="zone_a_r8_8" x="8.0" y="-20.8"/>
-    <xacro:big_shelf name="zone_a_r8_9" x="16.0" y="-20.8"/>
-    <xacro:big_shelf name="zone_a_r8_10" x="24.0" y="-20.8"/>
-    <xacro:big_shelf name="zone_a_r8_11" x="32.0" y="-20.8"/>
-    <xacro:big_shelf name="zone_a_r8_12" x="40.0" y="-20.8"/>
-    <xacro:big_shelf name="zone_a_r8_13" x="48.0" y="-20.8"/>
-    <xacro:big_shelf name="zone_a_r8_14" x="56.0" y="-20.8"/>
-    <xacro:big_shelf name="zone_a_r9_1" x="-56" y="-17.6"/>
-    <xacro:big_shelf name="zone_a_r9_2" x="-48.0" y="-17.6"/>
-    <xacro:big_shelf name="zone_a_r9_3" x="-40.0" y="-17.6"/>
-    <xacro:big_shelf name="zone_a_r9_4" x="-32.0" y="-17.6"/>
-    <xacro:big_shelf name="zone_a_r9_5" x="-24.0" y="-17.6"/>
-    <xacro:big_shelf name="zone_a_r9_6" x="-16.0" y="-17.6"/>
-    <xacro:big_shelf name="zone_a_r9_7" x="-8.0" y="-17.6"/>
-    <xacro:big_shelf name="zone_a_r9_8" x="8.0" y="-17.6"/>
-    <xacro:big_shelf name="zone_a_r9_9" x="16.0" y="-17.6"/>
-    <xacro:big_shelf name="zone_a_r9_10" x="24.0" y="-17.6"/>
-    <xacro:big_shelf name="zone_a_r9_11" x="32.0" y="-17.6"/>
-    <xacro:big_shelf name="zone_a_r9_12" x="40.0" y="-17.6"/>
-    <xacro:big_shelf name="zone_a_r9_13" x="48.0" y="-17.6"/>
-    <xacro:big_shelf name="zone_a_r9_14" x="56.0" y="-17.6"/>
-    <xacro:big_shelf name="zone_a_r10_1" x="-56" y="-16.4"/>
-    <xacro:big_shelf name="zone_a_r10_2" x="-48.0" y="-16.4"/>
-    <xacro:big_shelf name="zone_a_r10_3" x="-40.0" y="-16.4"/>
-    <xacro:big_shelf name="zone_a_r10_4" x="-32.0" y="-16.4"/>
-    <xacro:big_shelf name="zone_a_r10_5" x="-24.0" y="-16.4"/>
-    <xacro:big_shelf name="zone_a_r10_6" x="-16.0" y="-16.4"/>
-    <xacro:big_shelf name="zone_a_r10_7" x="-8.0" y="-16.4"/>
-    <xacro:big_shelf name="zone_a_r10_8" x="8.0" y="-16.4"/>
-    <xacro:big_shelf name="zone_a_r10_9" x="16.0" y="-16.4"/>
-    <xacro:big_shelf name="zone_a_r10_10" x="24.0" y="-16.4"/>
-    <xacro:big_shelf name="zone_a_r10_11" x="32.0" y="-16.4"/>
-    <xacro:big_shelf name="zone_a_r10_12" x="40.0" y="-16.4"/>
-    <xacro:big_shelf name="zone_a_r10_13" x="48.0" y="-16.4"/>
-    <xacro:big_shelf name="zone_a_r10_14" x="56.0" y="-16.4"/>
-    <xacro:big_shelf name="zone_a_r11_1" x="-56" y="-13.2"/>
-    <xacro:big_shelf name="zone_a_r11_2" x="-48.0" y="-13.2"/>
-    <xacro:big_shelf name="zone_a_r11_3" x="-40.0" y="-13.2"/>
-    <xacro:big_shelf name="zone_a_r11_4" x="-32.0" y="-13.2"/>
-    <xacro:big_shelf name="zone_a_r11_5" x="-24.0" y="-13.2"/>
-    <xacro:big_shelf name="zone_a_r11_6" x="-16.0" y="-13.2"/>
-    <xacro:big_shelf name="zone_a_r11_7" x="-8.0" y="-13.2"/>
-    <xacro:big_shelf name="zone_a_r11_8" x="8.0" y="-13.2"/>
-    <xacro:big_shelf name="zone_a_r11_9" x="16.0" y="-13.2"/>
-    <xacro:big_shelf name="zone_a_r11_10" x="24.0" y="-13.2"/>
-    <xacro:big_shelf name="zone_a_r11_11" x="32.0" y="-13.2"/>
-    <xacro:big_shelf name="zone_a_r11_12" x="40.0" y="-13.2"/>
-    <xacro:big_shelf name="zone_a_r11_13" x="48.0" y="-13.2"/>
-    <xacro:big_shelf name="zone_a_r11_14" x="56.0" y="-13.2"/>
-    <xacro:big_shelf name="zone_a_r12_1" x="-56" y="-12.0"/>
-    <xacro:big_shelf name="zone_a_r12_2" x="-48.0" y="-12.0"/>
-    <xacro:big_shelf name="zone_a_r12_3" x="-40.0" y="-12.0"/>
-    <xacro:big_shelf name="zone_a_r12_4" x="-32.0" y="-12.0"/>
-    <xacro:big_shelf name="zone_a_r12_5" x="-24.0" y="-12.0"/>
-    <xacro:big_shelf name="zone_a_r12_6" x="-16.0" y="-12.0"/>
-    <xacro:big_shelf name="zone_a_r12_7" x="-8.0" y="-12.0"/>
-    <xacro:big_shelf name="zone_a_r12_8" x="8.0" y="-12.0"/>
-    <xacro:big_shelf name="zone_a_r12_9" x="16.0" y="-12.0"/>
-    <xacro:big_shelf name="zone_a_r12_10" x="24.0" y="-12.0"/>
-    <xacro:big_shelf name="zone_a_r12_11" x="32.0" y="-12.0"/>
-    <xacro:big_shelf name="zone_a_r12_12" x="40.0" y="-12.0"/>
-    <xacro:big_shelf name="zone_a_r12_13" x="48.0" y="-12.0"/>
-    <xacro:big_shelf name="zone_a_r12_14" x="56.0" y="-12.0"/>
-    <xacro:big_shelf name="zone_a_r13_1" x="-56" y="-8.8"/>
-    <xacro:big_shelf name="zone_a_r13_2" x="-48.0" y="-8.8"/>
-    <xacro:big_shelf name="zone_a_r13_3" x="-40.0" y="-8.8"/>
-    <xacro:big_shelf name="zone_a_r13_4" x="-32.0" y="-8.8"/>
-    <xacro:big_shelf name="zone_a_r13_5" x="-24.0" y="-8.8"/>
-    <xacro:big_shelf name="zone_a_r13_6" x="-16.0" y="-8.8"/>
-    <xacro:big_shelf name="zone_a_r13_7" x="-8.0" y="-8.8"/>
-    <xacro:big_shelf name="zone_a_r13_8" x="8.0" y="-8.8"/>
-    <xacro:big_shelf name="zone_a_r13_9" x="16.0" y="-8.8"/>
-    <xacro:big_shelf name="zone_a_r13_10" x="24.0" y="-8.8"/>
-    <xacro:big_shelf name="zone_a_r13_11" x="32.0" y="-8.8"/>
-    <xacro:big_shelf name="zone_a_r13_12" x="40.0" y="-8.8"/>
-    <xacro:big_shelf name="zone_a_r13_13" x="48.0" y="-8.8"/>
-    <xacro:big_shelf name="zone_a_r13_14" x="56.0" y="-8.8"/>
-    <xacro:big_shelf name="zone_a_r14_1" x="-56" y="-7.6"/>
-    <xacro:big_shelf name="zone_a_r14_2" x="-48.0" y="-7.6"/>
-    <xacro:big_shelf name="zone_a_r14_3" x="-40.0" y="-7.6"/>
-    <xacro:big_shelf name="zone_a_r14_4" x="-32.0" y="-7.6"/>
-    <xacro:big_shelf name="zone_a_r14_5" x="-24.0" y="-7.6"/>
-    <xacro:big_shelf name="zone_a_r14_6" x="-16.0" y="-7.6"/>
-    <xacro:big_shelf name="zone_a_r14_7" x="-8.0" y="-7.6"/>
-    <xacro:big_shelf name="zone_a_r14_8" x="8.0" y="-7.6"/>
-    <xacro:big_shelf name="zone_a_r14_9" x="16.0" y="-7.6"/>
-    <xacro:big_shelf name="zone_a_r14_10" x="24.0" y="-7.6"/>
-    <xacro:big_shelf name="zone_a_r14_11" x="32.0" y="-7.6"/>
-    <xacro:big_shelf name="zone_a_r14_12" x="40.0" y="-7.6"/>
-    <xacro:big_shelf name="zone_a_r14_13" x="48.0" y="-7.6"/>
-    <xacro:big_shelf name="zone_a_r14_14" x="56.0" y="-7.6"/>
+    <xacro:big_shelf name="zone_a_r1_1" x="-54.0" y="-37.2"/>
+    <xacro:big_shelf name="zone_a_r1_2" x="-46.0" y="-37.2"/>
+    <xacro:big_shelf name="zone_a_r1_3" x="-38.0" y="-37.2"/>
+    <xacro:big_shelf name="zone_a_r1_4" x="-30.0" y="-37.2"/>
+    <xacro:big_shelf name="zone_a_r1_5" x="-22.0" y="-37.2"/>
+    <xacro:big_shelf name="zone_a_r1_6" x="-14.0" y="-37.2"/>
+    <xacro:big_shelf name="zone_a_r1_7" x="-6.0" y="-37.2"/>
+    <xacro:big_shelf name="zone_a_r1_8" x="10.0" y="-37.2"/>
+    <xacro:big_shelf name="zone_a_r1_9" x="18.0" y="-37.2"/>
+    <xacro:big_shelf name="zone_a_r1_10" x="26.0" y="-37.2"/>
+    <xacro:big_shelf name="zone_a_r1_11" x="34.0" y="-37.2"/>
+    <xacro:big_shelf name="zone_a_r1_12" x="42.0" y="-37.2"/>
+    <xacro:big_shelf name="zone_a_r1_13" x="50.0" y="-37.2"/>
+    <xacro:big_shelf name="zone_a_r1_14" x="58.0" y="-37.2"/>
+    <xacro:big_shelf name="zone_a_r2_1" x="-54.0" y="-36.0"/>
+    <xacro:big_shelf name="zone_a_r2_2" x="-46.0" y="-36.0"/>
+    <xacro:big_shelf name="zone_a_r2_3" x="-38.0" y="-36.0"/>
+    <xacro:big_shelf name="zone_a_r2_4" x="-30.0" y="-36.0"/>
+    <xacro:big_shelf name="zone_a_r2_5" x="-22.0" y="-36.0"/>
+    <xacro:big_shelf name="zone_a_r2_6" x="-14.0" y="-36.0"/>
+    <xacro:big_shelf name="zone_a_r2_7" x="-6.0" y="-36.0"/>
+    <xacro:big_shelf name="zone_a_r2_8" x="10.0" y="-36.0"/>
+    <xacro:big_shelf name="zone_a_r2_9" x="18.0" y="-36.0"/>
+    <xacro:big_shelf name="zone_a_r2_10" x="26.0" y="-36.0"/>
+    <xacro:big_shelf name="zone_a_r2_11" x="34.0" y="-36.0"/>
+    <xacro:big_shelf name="zone_a_r2_12" x="42.0" y="-36.0"/>
+    <xacro:big_shelf name="zone_a_r2_13" x="50.0" y="-36.0"/>
+    <xacro:big_shelf name="zone_a_r2_14" x="58.0" y="-36.0"/>
+    <xacro:big_shelf name="zone_a_r3_1" x="-54.0" y="-32.8"/>
+    <xacro:big_shelf name="zone_a_r3_2" x="-46.0" y="-32.8"/>
+    <xacro:big_shelf name="zone_a_r3_3" x="-38.0" y="-32.8"/>
+    <xacro:big_shelf name="zone_a_r3_4" x="-30.0" y="-32.8"/>
+    <xacro:big_shelf name="zone_a_r3_5" x="-22.0" y="-32.8"/>
+    <xacro:big_shelf name="zone_a_r3_6" x="-14.0" y="-32.8"/>
+    <xacro:big_shelf name="zone_a_r3_7" x="-6.0" y="-32.8"/>
+    <xacro:big_shelf name="zone_a_r3_8" x="10.0" y="-32.8"/>
+    <xacro:big_shelf name="zone_a_r3_9" x="18.0" y="-32.8"/>
+    <xacro:big_shelf name="zone_a_r3_10" x="26.0" y="-32.8"/>
+    <xacro:big_shelf name="zone_a_r3_11" x="34.0" y="-32.8"/>
+    <xacro:big_shelf name="zone_a_r3_12" x="42.0" y="-32.8"/>
+    <xacro:big_shelf name="zone_a_r3_13" x="50.0" y="-32.8"/>
+    <xacro:big_shelf name="zone_a_r3_14" x="58.0" y="-32.8"/>
+    <xacro:big_shelf name="zone_a_r4_1" x="-54.0" y="-31.6"/>
+    <xacro:big_shelf name="zone_a_r4_2" x="-46.0" y="-31.6"/>
+    <xacro:big_shelf name="zone_a_r4_3" x="-38.0" y="-31.6"/>
+    <xacro:big_shelf name="zone_a_r4_4" x="-30.0" y="-31.6"/>
+    <xacro:big_shelf name="zone_a_r4_5" x="-22.0" y="-31.6"/>
+    <xacro:big_shelf name="zone_a_r4_6" x="-14.0" y="-31.6"/>
+    <xacro:big_shelf name="zone_a_r4_7" x="-6.0" y="-31.6"/>
+    <xacro:big_shelf name="zone_a_r4_8" x="10.0" y="-31.6"/>
+    <xacro:big_shelf name="zone_a_r4_9" x="18.0" y="-31.6"/>
+    <xacro:big_shelf name="zone_a_r4_10" x="26.0" y="-31.6"/>
+    <xacro:big_shelf name="zone_a_r4_11" x="34.0" y="-31.6"/>
+    <xacro:big_shelf name="zone_a_r4_12" x="42.0" y="-31.6"/>
+    <xacro:big_shelf name="zone_a_r4_13" x="50.0" y="-31.6"/>
+    <xacro:big_shelf name="zone_a_r4_14" x="58.0" y="-31.6"/>
+    <xacro:big_shelf name="zone_a_r5_1" x="-54.0" y="-28.4"/>
+    <xacro:big_shelf name="zone_a_r5_2" x="-46.0" y="-28.4"/>
+    <xacro:big_shelf name="zone_a_r5_3" x="-38.0" y="-28.4"/>
+    <xacro:big_shelf name="zone_a_r5_4" x="-30.0" y="-28.4"/>
+    <xacro:big_shelf name="zone_a_r5_5" x="-22.0" y="-28.4"/>
+    <xacro:big_shelf name="zone_a_r5_6" x="-14.0" y="-28.4"/>
+    <xacro:big_shelf name="zone_a_r5_7" x="-6.0" y="-28.4"/>
+    <xacro:big_shelf name="zone_a_r5_8" x="10.0" y="-28.4"/>
+    <xacro:big_shelf name="zone_a_r5_9" x="18.0" y="-28.4"/>
+    <xacro:big_shelf name="zone_a_r5_10" x="26.0" y="-28.4"/>
+    <xacro:big_shelf name="zone_a_r5_11" x="34.0" y="-28.4"/>
+    <xacro:big_shelf name="zone_a_r5_12" x="42.0" y="-28.4"/>
+    <xacro:big_shelf name="zone_a_r5_13" x="50.0" y="-28.4"/>
+    <xacro:big_shelf name="zone_a_r5_14" x="58.0" y="-28.4"/>
+    <xacro:big_shelf name="zone_a_r6_1" x="-54.0" y="-27.2"/>
+    <xacro:big_shelf name="zone_a_r6_2" x="-46.0" y="-27.2"/>
+    <xacro:big_shelf name="zone_a_r6_3" x="-38.0" y="-27.2"/>
+    <xacro:big_shelf name="zone_a_r6_4" x="-30.0" y="-27.2"/>
+    <xacro:big_shelf name="zone_a_r6_5" x="-22.0" y="-27.2"/>
+    <xacro:big_shelf name="zone_a_r6_6" x="-14.0" y="-27.2"/>
+    <xacro:big_shelf name="zone_a_r6_7" x="-6.0" y="-27.2"/>
+    <xacro:big_shelf name="zone_a_r6_8" x="10.0" y="-27.2"/>
+    <xacro:big_shelf name="zone_a_r6_9" x="18.0" y="-27.2"/>
+    <xacro:big_shelf name="zone_a_r6_10" x="26.0" y="-27.2"/>
+    <xacro:big_shelf name="zone_a_r6_11" x="34.0" y="-27.2"/>
+    <xacro:big_shelf name="zone_a_r6_12" x="42.0" y="-27.2"/>
+    <xacro:big_shelf name="zone_a_r6_13" x="50.0" y="-27.2"/>
+    <xacro:big_shelf name="zone_a_r6_14" x="58.0" y="-27.2"/>
+    <xacro:big_shelf name="zone_a_r7_1" x="-54.0" y="-22.0"/>
+    <xacro:big_shelf name="zone_a_r7_2" x="-46.0" y="-22.0"/>
+    <xacro:big_shelf name="zone_a_r7_3" x="-38.0" y="-22.0"/>
+    <xacro:big_shelf name="zone_a_r7_4" x="-30.0" y="-22.0"/>
+    <xacro:big_shelf name="zone_a_r7_5" x="-22.0" y="-22.0"/>
+    <xacro:big_shelf name="zone_a_r7_6" x="-14.0" y="-22.0"/>
+    <xacro:big_shelf name="zone_a_r7_7" x="-6.0" y="-22.0"/>
+    <xacro:big_shelf name="zone_a_r7_8" x="10.0" y="-22.0"/>
+    <xacro:big_shelf name="zone_a_r7_9" x="18.0" y="-22.0"/>
+    <xacro:big_shelf name="zone_a_r7_10" x="26.0" y="-22.0"/>
+    <xacro:big_shelf name="zone_a_r7_11" x="34.0" y="-22.0"/>
+    <xacro:big_shelf name="zone_a_r7_12" x="42.0" y="-22.0"/>
+    <xacro:big_shelf name="zone_a_r7_13" x="50.0" y="-22.0"/>
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