Commit message: Nav2 at least brings up :-)
Signed-off-by: SteveMacenski <stevenmacenski@gmail.com>

File: opennav_benchmark_robot/urdf/benchmark_robot.sdf.xacro (robot description, xacro)
@@ -10,9 +10,9 @@
     <xacro:property name="robot_visibility_flags" value="0xFFFE"/>
     <xacro:property name="lidar_visibility_mask" value="0x0001"/>
-    <!-- Base footprint link (ground reference) -->
-    <link name="base_footprint"/>
     <!-- ============ CHASSIS (rounded mesh) ============ -->
     <link name="base_link">
-      <pose relative_to="base_footprint">0 0 0.25 0 0 0</pose>
+    <!-- Base footprint link (ground reference) -->
+    <link name="base_footprint">
+      <pose relative_to="base_link">0 0 -0.25 0 0 0</pose>
       <inertial>
         <mass>200.0</mass>

File: opennav_benchmark_robot/urdf/benchmark_robot.urdf.xacro (robot description, xacro)
@@ -71,7 +71,7 @@
   </link>
   <joint name="base_joint" type="fixed">
-    <parent link="base_footprint"/>
-    <child link="base_link"/>
-    <origin xyz="0 0 ${chassis_z_offset}" rpy="0 0 0"/>
+    <parent link="base_link"/>
+    <child link="base_footprint"/>
+    <origin xyz="0 0 ${-chassis_z_offset}" rpy="0 0 0"/>
   </joint>
   <!-- ============ DRIVE WHEELS ============ -->

Commit message: fixing frame issue
Signed-off-by: SteveMacenski <stevenmacenski@gmail.com>

File: opennav_benchmark_robot/urdf/benchmark_robot.sdf.xacro (robot description, xacro)
@@ -12,31 +12,32 @@
     <!-- ============ CHASSIS (rounded mesh) ============ -->
     <link name="base_link">
+      <inertial>
+        <mass>200.0</mass>
+        <inertia>
+          <ixx>12.08</ixx><ixy>0</ixy><ixz>0</ixz>
+          <iyy>26.17</iyy><iyz>0</iyz>
+          <izz>35.33</izz>
+        </inertia>
+      </inertial>
+      <visual name="chassis_visual">
+        <visibility_flags>${robot_visibility_flags}</visibility_flags>
+        <pose>0 0 -0.25 1.5708 0 -1.5708</pose>
+        <geometry>
+          <mesh><uri>package://opennav_benchmark_robot/meshes/Forklift_agv_01.obj</uri></mesh>
+        </geometry>
+      </visual>
+      <collision name="chassis_collision">
+        <geometry>
+          <box><size>1.2 0.8 0.3</size></box>
+        </geometry>
+      </collision>
+    </link>
     <!-- Base footprint link (ground reference) -->
     <link name="base_footprint">
       <pose relative_to="base_link">0 0 -0.25 0 0 0</pose>
-      <inertial>
-        <mass>200.0</mass>
-        <inertia>
-          <ixx>12.08</ixx><ixy>0</ixy><ixz>0</ixz>
-          <iyy>26.17</iyy><iyz>0</iyz>
-          <izz>35.33</izz>
-        </inertia>
-      </inertial>
-      <visual name="chassis_visual">
-        <visibility_flags>${robot_visibility_flags}</visibility_flags>
-        <pose>0 0 -0.25 1.5708 0 -1.5708</pose>
-        <geometry>
-          <mesh><uri>package://opennav_benchmark_robot/meshes/Forklift_agv_01.obj</uri></mesh>
-        </geometry>
-      </visual>
-      <collision name="chassis_collision">
-        <geometry>
-          <box><size>1.2 0.8 0.3</size></box>
-        </geometry>
-      </collision>
     </link>
     <joint name="base_joint" type="fixed">
-      <parent>base_footprint</parent>
-      <child>base_link</child>
+      <parent>base_link</parent>
+      <child>base_footprint</child>
     </joint>
     <!-- ============ DRIVE WHEELS ============ -->

Commit message: working initial testing, at non-realtime
Signed-off-by: SteveMacenski <stevenmacenski@gmail.com>

File: opennav_benchmark_robot/urdf/benchmark_robot.sdf.xacro (robot description, xacro)
@@ -234,5 +234,5 @@
           </scan>
           <range>
-            <min>0.3</min>
+            <min>1.0</min>
             <max>30.0</max>
             <resolution>0.01</resolution>
@@ -293,5 +293,5 @@
           </scan>
           <range>
-            <min>0.3</min>
+            <min>1.0</min>
             <max>30.0</max>
             <resolution>0.01</resolution>
@@ -337,4 +337,5 @@
         <update_rate>10</update_rate>
         <lidar>
+          <visibility_mask>${lidar_visibility_mask}</visibility_mask>
           <scan>
             <horizontal>
@@ -352,5 +353,5 @@
           </scan>
           <range>
-            <min>0.3</min>
+            <min>1.0</min>
             <max>30.0</max>
             <resolution>0.01</resolution>
@@ -400,6 +401,6 @@
               <samples>720</samples>
               <resolution>1</resolution>
-              <min_angle>-2.356</min_angle>
-              <max_angle>2.356</max_angle>
+              <min_angle>-2.0944</min_angle>  <!-- 270 - 15 deg for robot self collision filter clearance-->
+              <max_angle>2.0944</max_angle>
             </horizontal>
             <vertical>
@@ -458,6 +459,6 @@
               <samples>720</samples>
               <resolution>1</resolution>
-              <min_angle>-2.356</min_angle>
-              <max_angle>2.356</max_angle>
+              <min_angle>-2.0944</min_angle> <!-- 270 - 15 deg for robot self collision filter clearance -->
+              <max_angle>2.0944</max_angle>
             </horizontal>
             <vertical>

File: opennav_benchmark_sim/worlds/benchmark_warehouse.sdf.xacro (robot description, xacro)
@@ -4,8 +4,8 @@
   <world name="benchmark_warehouse">
     <!-- Physics -->
-    <physics name="5ms" type="bullet">
-      <max_step_size>0.005</max_step_size>
-      <real_time_update_rate>500.0</real_time_update_rate>
-      <real_time_factor>1.0</real_time_factor>
+    <physics name="tpe" type="tpe">
+      <engine>
+        <filename>gz-physics-tpe-plugin</filename>
+      </engine>
     </physics>
     <!-- Plugins -->
@@ -193,4 +193,13 @@
       <include>
         <uri>https://fuel.gazebosim.org/1.0/OpenRobotics/models/Casual female</uri>
+        <name>${name}</name>
+        <pose>${x} ${y} 0 0 0 ${yaw}</pose>
+        <static>true</static>
+      </include>
+    </xacro:macro>
+    <!-- Charging station (Fuel model from MovAi) -->
+    <xacro:macro name="charging_station" params="name x y yaw">
+      <include>
+        <uri>https://fuel.gazebosim.org/1.0/MovAi/models/Tugbot-charging-station</uri>
         <name>${name}</name>
         <pose>${x} ${y} 0 0 0 ${yaw}</pose>
@@ -1648,4 +1657,6 @@
     <xacro:forklift name="spill2_forklift" x="-25.6955" y="-10.5044" yaw="3.0"/>
     <xacro:person name="spill2_p1" x="-24.5" y="-14.200000000000001" yaw="3.14"/>
+    <!-- Charging station -->
+    <xacro:charging_station name="charging_station_1" x="63.7013" y="35.9283" yaw="0"/>
   </world>
 </sdf>
