Commit message: adding the vlm camera to simulation
Signed-off-by: SteveMacenski <stevenmacenski@gmail.com>

File: opennav_benchmark_simulation/opennav_benchmark_robot/urdf/benchmark_robot.sdf.xacro (robot description, xacro)
@@ -488,4 +488,37 @@
       <parent>base_link</parent>
       <child>lidar_2d_front_right_link</child>
+    </joint>
+    <!-- ============ CAMERA (between 2D lidars) ============ -->
+    <link name="camera_front_link">
+      <pose relative_to="base_link">-0.65 0 0.60 0 0 3.14159</pose>
+      <inertial>
+        <mass>0.1</mass>
+        <inertia>
+          <ixx>0.00001</ixx><ixy>0</ixy><ixz>0</ixz>
+          <iyy>0.00001</iyy><iyz>0</iyz>
+          <izz>0.00001</izz>
+        </inertia>
+      </inertial>
+      <sensor name="camera_front_sensor" type="camera">
+        <always_on>true</always_on>
+        <update_rate>5</update_rate>
+        <camera>
+          <horizontal_fov>1.047</horizontal_fov>
+          <image>
+            <width>640</width>
+            <height>480</height>
+          </image>
+          <clip>
+            <near>0.1</near>
+            <far>100.0</far>
+          </clip>
+        </camera>
+        <topic>${ns}/camera_front/image</topic>
+        <gz_frame_id>camera_front_link</gz_frame_id>
+      </sensor>
+    </link>
+    <joint name="camera_front_joint" type="fixed">
+      <parent>base_link</parent>
+      <child>camera_front_link</child>
     </joint>
     <!-- ============ DEPTH CAMERAS (Orbbec Gemini 335 on chassis faces) ============ -->

Commit message: Simulation and behavioral improvements using VLM and docking server
Signed-off-by: SteveMacenski <stevenmacenski@gmail.com>

File: opennav_benchmark_simulation/opennav_benchmark_robot/urdf/benchmark_robot.sdf.xacro (robot description, xacro)
@@ -23,5 +23,5 @@
       <visual name="chassis_visual">
         <visibility_flags>${robot_visibility_flags}</visibility_flags>
-        <pose>0 0 -0.25 1.5708 0 -1.5708</pose>
+        <pose>0 0 -0.25 1.5708 0 1.5708</pose>
         <geometry>
           <mesh><uri>package://opennav_benchmark_robot/meshes/Forklift_agv_01.obj</uri></mesh>
@@ -155,8 +155,8 @@
       </joint>
     </xacro:macro>
-    <xacro:caster_sdf name="rear_left" x="0.45" y="0.30"/>
-    <xacro:caster_sdf name="rear_right" x="0.45" y="-0.30"/>
-    <xacro:caster_sdf name="front_left" x="-0.45" y="0.30"/>
-    <xacro:caster_sdf name="front_right" x="-0.45" y="-0.30"/>
+    <xacro:caster_sdf name="front_left" x="0.45" y="0.30"/>
+    <xacro:caster_sdf name="front_right" x="0.45" y="-0.30"/>
+    <xacro:caster_sdf name="rear_left" x="-0.45" y="0.30"/>
+    <xacro:caster_sdf name="rear_right" x="-0.45" y="-0.30"/>
     <!-- ============ IMU ============ -->
     <link name="imu_link">
@@ -196,5 +196,5 @@
     <!-- Center: 360deg, 32ch -->
     <link name="lidar_3d_center_link">
-      <pose relative_to="base_link">0.10 0 0.825 0 0 0</pose>
+      <pose relative_to="base_link">-0.10 0 0.825 0 0 3.14159</pose>
       <inertial>
         <mass>0.5</mass>
@@ -255,5 +255,5 @@
     <!-- Top: on tower surface, in front of center lidar -->
     <link name="lidar_3d_top_link">
-      <pose relative_to="base_link">0.35 0 2.195 0 0 0</pose>
+      <pose relative_to="base_link">-0.35 0 2.195 0 0 3.14159</pose>
       <inertial>
         <mass>0.5</mass>
@@ -314,5 +314,5 @@
     <!-- Front-right: 16ch, tilted down 15deg -->
     <link name="lidar_3d_tilted_link">
-      <pose relative_to="base_link">0.10 0 1.845 0.7854 0 1.5708</pose>
+      <pose relative_to="base_link">-0.10 0 1.845 0.7854 0 -1.5708</pose>
       <inertial>
         <mass>0.5</mass>
@@ -374,5 +374,5 @@
     <!-- ============ 2D LIDARS (SICK TiM781 on chassis corners) ============ -->
     <link name="lidar_2d_front_left_link">
-      <pose relative_to="base_link">-0.50 0.40 0.60 0 0 2.356</pose>
+      <pose relative_to="base_link">0.50 0.40 0.60 0 0 0.7854</pose>
       <inertial>
         <mass>0.4</mass>
@@ -432,5 +432,5 @@
     </joint>
     <link name="lidar_2d_front_right_link">
-      <pose relative_to="base_link">-0.50 -0.40 0.60 0 0 -2.356</pose>
+      <pose relative_to="base_link">0.50 -0.40 0.60 0 0 -0.7854</pose>
       <inertial>
         <mass>0.4</mass>
@@ -491,5 +491,5 @@
     <!-- ============ CAMERA (between 2D lidars) ============ -->
     <link name="camera_front_link">
-      <pose relative_to="base_link">-0.65 0 0.60 0 0 3.14159</pose>
+      <pose relative_to="base_link">0.65 0 0.60 0 0 0</pose>
       <inertial>
         <mass>0.1</mass>
@@ -567,7 +567,7 @@
       </joint>
     </xacro:macro>
-    <xacro:camera_sdf name="camera_rear" x="0.235" y="0" z="0.175" pitch="0" yaw="0"/>
-    <xacro:camera_sdf name="camera_front_left" x="-0.63" y="0.20" z="0.10" pitch="0.2618" yaw="${3.14159 + 0.5245}"/>
-    <xacro:camera_sdf name="camera_front_right" x="-0.63" y="-0.20" z="0.10" pitch="0.2618" yaw="${3.14159 - 0.5245}"/>
+    <xacro:camera_sdf name="camera_rear" x="-0.235" y="0" z="0.175" pitch="0" yaw="3.14159"/>
+    <xacro:camera_sdf name="camera_front_left" x="0.63" y="0.20" z="0.10" pitch="0.2618" yaw="-0.5245"/>
+    <xacro:camera_sdf name="camera_front_right" x="0.63" y="-0.20" z="0.10" pitch="0.2618" yaw="0.5245"/>
     <!-- ============ PLUGINS ============ -->
     <plugin filename="gz-sim-diff-drive-system" name="gz::sim::systems::DiffDrive">

File: opennav_benchmark_simulation/opennav_benchmark_robot/urdf/benchmark_robot.urdf.xacro (robot description, xacro)
@@ -58,5 +58,5 @@
   <link name="base_link">
     <visual>
-      <origin xyz="0 0 -0.25" rpy="1.5708 0 -1.5708"/>
+      <origin xyz="0 0 -0.25" rpy="1.5708 0 1.5708"/>
       <geometry>
         <mesh filename="package://opennav_benchmark_robot/meshes/Forklift_agv_01.obj"/>
@@ -124,8 +124,8 @@
     </joint>
   </xacro:macro>
-  <xacro:caster_wheel name="rear_left" x="0.45" y="0.30"/>
-  <xacro:caster_wheel name="rear_right" x="0.45" y="-0.30"/>
-  <xacro:caster_wheel name="front_left" x="-0.45" y="0.30"/>
-  <xacro:caster_wheel name="front_right" x="-0.45" y="-0.30"/>
+  <xacro:caster_wheel name="front_left" x="0.45" y="0.30"/>
+  <xacro:caster_wheel name="front_right" x="0.45" y="-0.30"/>
+  <xacro:caster_wheel name="rear_left" x="-0.45" y="0.30"/>
+  <xacro:caster_wheel name="rear_right" x="-0.45" y="-0.30"/>
   <!-- ============ IMU ============ -->
   <link name="imu_link">
@@ -160,5 +160,5 @@
     <parent link="base_link"/>
     <child link="lidar_3d_center_link"/>
-    <origin xyz="0.10 0 0.825" rpy="0 0 0"/>
+    <origin xyz="-0.10 0 0.825" rpy="0 0 ${pi}"/>
   </joint>
   <!-- Top: on tower surface, in front of center lidar -->
@@ -181,5 +181,5 @@
     <parent link="base_link"/>
     <child link="lidar_3d_top_link"/>
-    <origin xyz="0.35 0 2.195" rpy="0 0 0"/>
+    <origin xyz="-0.35 0 2.195" rpy="0 0 ${pi}"/>
   </joint>
   <!-- Tilted: 16ch, pitched 270deg -->
@@ -202,5 +202,5 @@
     <parent link="base_link"/>
     <child link="lidar_3d_tilted_link"/>
-    <origin xyz="0.10 0 1.845" rpy="${pi/4} 0 ${pi/2}"/>
+    <origin xyz="-0.10 0 1.845" rpy="${pi/4} 0 ${-pi/2}"/>
   </joint>
   <!-- ============ 2D LIDARS (SICK TiM781 on chassis corners) ============ -->
@@ -227,6 +227,6 @@
     </joint>
   </xacro:macro>
-  <xacro:lidar_2d name="lidar_2d_front_left" x="-0.50" y="0.40" yaw="${3*pi/4}"/>
-  <xacro:lidar_2d name="lidar_2d_front_right" x="-0.50" y="-0.40" yaw="${-3*pi/4}"/>
+  <xacro:lidar_2d name="lidar_2d_front_left" x="0.50" y="0.40" yaw="${pi/4}"/>
+  <xacro:lidar_2d name="lidar_2d_front_right" x="0.50" y="-0.40" yaw="${-pi/4}"/>
   <!-- ============ DEPTH CAMERAS (Orbbec Gemini 335) ============ -->
   <xacro:macro name="depth_camera" params="name x y z pitch yaw">
@@ -258,6 +258,6 @@
     </joint>
   </xacro:macro>
-  <xacro:depth_camera name="camera_rear" x="0.235" y="0" z="0.175" pitch="0" yaw="0"/>
-  <xacro:depth_camera name="camera_front_left" x="-0.63" y="0.20" z="0.10" pitch="${pi/12}" yaw="${pi + 0.5245}"/>
-  <xacro:depth_camera name="camera_front_right" x="-0.63" y="-0.20" z="0.10" pitch="${pi/12}" yaw="${pi - 0.5245}"/>
+  <xacro:depth_camera name="camera_rear" x="-0.235" y="0" z="0.175" pitch="0" yaw="${pi}"/>
+  <xacro:depth_camera name="camera_front_left" x="0.63" y="0.20" z="0.10" pitch="${pi/12}" yaw="${-0.5245}"/>
+  <xacro:depth_camera name="camera_front_right" x="0.63" y="-0.20" z="0.10" pitch="${pi/12}" yaw="${0.5245}"/>
 </robot>
